File: hardware/v0.1/1.brd (EAGLE design)
At the start: 80 x 40 mm, 84 parts, among them IC1 FP6291, IC2 TSOP34830, IC3 TSOP34830, IC4 STM32F10XCXT6, IC6 TM1809, Q1 8050, Q2 8050, U1 74LVC1G08SE-7, Y1 8m

Commit message: start wiring
Parts:
- removed L1: 4.7uh, SparkFun-Passives:IHLP4040DZ
- added L3: 4.7uh, SparkFun-Passives:CR75_V2
- C1: value 100nf -> 100uf; device SparkFun-Passives:0402-CAP -> SparkFun-Capacitors:EIA6032
- C10: value 4.7uf -> 1uf; device SparkFun-Passives:0603-CAP -> SparkFun-Passives:0402-CAP
- C19: device SparkFun-Passives:0402-CAP -> SparkFun-Passives:0603-CAP
- C2, C4: value 10uf -> 100nf; device SparkFun-Passives:0402-CAP -> SparkFun-Passives:0603-CAP
- C20: value 4.7uf -> 100nf; device SparkFun-Passives:0402-CAP -> SparkFun-Passives:0603-CAP
- C21: value 100uf -> 100nf; device SparkFun-Capacitors:EIA6032 -> SparkFun-Passives:0402-CAP
- C22: value 100nf -> 4.7uf; device SparkFun-Passives:0603-CAP -> SparkFun-Passives:0402-CAP
- C23: value 1uf -> 4.7uf
- C24: value 100nf -> 4.7uf
- C3: value 10uf -> 1uf; device SparkFun-Passives:0402-CAP -> SparkFun-Passives:0603-CAP
- C6, C7: value 100nf -> 10uf; device SparkFun-Passives:0603-CAP -> SparkFun-Passives:0402-CAP
- C8: value 1uf -> 10uf
- C9: value 4.7uf -> 100nf; device SparkFun-Passives:0603-CAP -> SparkFun-Passives:0402-CAP
- D1: device SparkFun-DiscreteSemi:SMB-DIODE -> SparkFun-DiscreteSemi:SMA-DIODE
- IC2: value TSOP34830 -> TM1809; device vishay-1:TSOP348 -> eagle_lib_lishen:SOP-14
- IC3: value TSOP34830 -> STM32F10XCXT6; device vishay-1:TSOP348 -> stm32:TQFP48
- IC4: value STM32F10XCXT6 -> (none); device stm32:TQFP48 -> SparkFun-PowerIC:SOT23-3
- IC5: value (none) -> TSOP34830; device SparkFun-PowerIC:SOT23-3 -> vishay-1:TSOP348
- IC6: value TM1809 -> TSOP34830; device eagle_lib_lishen:SOP-14 -> vishay-1:TSOP348
- LED1: value IR -> LED-TRICOLOR-5050NO_IC; device SparkFun-LED:LED5MM -> SparkFun-LED:LED-TRICOLOR-5050
- LED2: value LED-TRICOLOR-5050NO_IC -> IR; device SparkFun-LED:LED-TRICOLOR-5050 -> SparkFun-LED:LED5MM
- R10: value 1m -> 2.2K
- R11: value 470R -> 51; device SparkFun-Passives:0603-RES -> SparkFun-Resistors:1206
- R12, R15: value 470R -> 10K
- R13, R14: value 470R -> 220R
- R17: value 470R -> 110K
- R18: value 470R -> 15K
- R2: value 51R -> 180R
- R20: value 100R -> 470R
- R21, R4: value 10K -> 470R
- R22, R23: value 220R -> 470R
- R24: value 220R -> 10K
- R25: value 220R -> 1m
- R26: value 180R -> 100R
- R27: value 2.2K -> 100R
- R3: value 47k -> 470R
- R5: value 110K -> 470R
- R6: value 15K -> 220R
- R7: value 100R -> 220R
- R8: value 100R -> 47k
- R9: value 10K -> 100R
- S3: device digital-toy:SWITCH-SPDT-AM#6 -> switch-dil:DIP03YL
- S4: device switch-dil:DIP03YL -> digital-toy:SWITCH-SPDT-AM#6
- Y1: value 8m -> 8M; device SparkFun-FreqCtrl:HC49US -> SparkFun-FreqCtrl:CRYSTAL-TXC-7A
- moved SG1 254.6 mm to (47.0, 43.0), turned to 180 degrees
- moved R26 248.9 mm to (9.00, 47.0)
- moved R25 239.8 mm to (57.0, 19.0)
- moved R24 230.7 mm to (54.7, 11.5), turned to 180 degrees
- moved Q2 223.0 mm to (7.00, 22.0), turned to 90 degrees
- moved R27 217.0 mm to (14.1, 2.95), turned to 180 degrees
- moved R23 214.7 mm to (33.0, 13.0)
- moved R18 214.4 mm to (69.0, 36.0), turned to 90 degrees
- moved R22 213.9 mm to (33.0, 15.0)
- moved R21 213.2 mm to (33.0, 17.0)
- moved R17 212.4 mm to (67.0, 38.0), flipped to the bottom
- moved R20 209.8 mm to (33.0, 19.0)
- moved LED8 199.0 mm to (29.0, 13.0), turned to 90 degrees
- moved LED7 195.9 mm to (29.0, 15.0), turned to 90 degrees
- moved LED6 193.0 mm to (29.0, 17.0), turned to 90 degrees
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Connections:
- removed net N$43 (its old number): Q2.1, R27.1
- new net N$9: Q2.1, R10.1
- net 3.3V: now also C21.1, C22.1, IC3.24, IC3.36, IC3.48, IC3.7, IC3.9; no longer C19.1, C20.1, IC4.24, IC4.36, IC4.48, IC4.7, IC4.9
- net 5V: now also C1.P$1, C10.1, C2.1, C7.1, C9.1, IC4.3, R22.2, R23.2, R27.2, R3.2, R4.2, R9.2; no longer C21.P$1, C22.1, C23.1, C24.1, C5.1, IC5.3, R13.2, R14.2, R15.2, R18.2, R7.2, R8.2
- net BUZZER: now also R1.2; no longer R27.2
- net DIP_SW1: now also S3.1; no longer S4.1
- net DIP_SW2: now also S3.2; no longer S4.2
- net DIP_SW3: now also S3.3; no longer S4.3
- net GND: now also C1.P$2, C21.2, IC2.7, IC3.23, IC3.35, IC3.47, IC3.8, IC4.1, IC5.2, IC6.2, R15.2, R18.1, R24.1, R8.1, S3.4, S3.5, S3.6; no longer C1.2, C21.P$2, IC2.2, IC3.2, IC4.23, IC4.35, IC4.47, IC4.8, IC5.1, IC6.7, R3.1, R4.2, R6.1, R9.1, S4.4, S4.5, S4.6
- net I2C_SCL: now also R13.2; no longer R24.2
- net I2C_SDA: now also R14.2; no longer R25.2
- net IR_RECEIVE1: now also IC5.1; no longer IC2.1
- net IR_RECEIVE2: now also IC6.1; no longer IC3.1
- net LED_CTRL: now also IC2.14, R12.1; no longer IC6.14, R21.1
- net N$1: now also IC3.20, R15.1; no longer IC4.20, R4.1
- net N$10: now also S4.3; no longer S3.3
- net N$11: now also C19.1, C23.1, IC5.3, R26.1; no longer C6.1, C9.1, IC2.3, R7.1
- net N$12: now also C20.1, C24.1, IC6.3, R27.1; no longer C10.1, C7.1, IC3.3, R8.1
- net N$13: now also IC2.4, LED1.5; no longer IC6.4, LED2.5
- net N$14: now also LED2.A, R11.1; no longer LED1.A, R2.1
- net N$15: now also IC2.5, LED1.6; no longer IC6.5, LED2.6
- net N$16: now also IC2.6, LED1.4; no longer IC6.6, LED2.4
- net N$17: now also LED1.2, R5.1; no longer LED2.2, R11.1
- net N$18: now also LED1.1, R4.1; no longer LED2.1, R12.1
- net N$19: now also LED1.3, R3.1; no longer LED2.3, R13.1
- net N$2: now also IC3.44, R24.2; no longer IC4.44, R9.2
- net N$20: now also C5.1, C6.1, L3.P$1; no longer C1.1, C2.1, L1.P$1
- net N$21: now also IC2.13; no longer IC6.13
- net N$22: now also L3.P$2; no longer L1.P$2
- net N$23: now also R8.2; no longer R3.2
- net N$24: now also R16.1; no longer R14.1
- net N$25: now also R17.1, R18.2; no longer R5.1, R6.2
- net N$26: now also R19.1; no longer R15.1
- net N$27: now also IC2.12; no longer IC6.12
- net N$28: now also IC2.11; no longer IC6.11
- net N$29: now also IC2.10; no longer IC6.10
- net N$3: now also IC3.5, R25.2, Y1.P$2; no longer IC4.5, R10.2, Y1.2
- net N$30: now also IC2.9; no longer IC6.9
- net N$31: now also IC2.8; no longer IC6.8
- net N$32: now also R20.1; no longer R16.1
- net N$33: now also R21.1; no longer R17.1
- net N$34: now also R22.1; no longer R18.1
- net N$35: now also R23.1; no longer R19.1
- net N$36: now also IC2.1, R9.1; no longer IC6.1, R20.1
- net N$37: now also IC3.30, R6.2; no longer IC4.30, R22.2
- net N$38: now also IC3.31, R7.2; no longer IC4.31, R23.2
- net N$39: now also IC3.43, R14.1; no longer IC4.43, R25.1
- net N$4: now also IC3.6, R25.1, Y1.P$1; no longer IC4.6, R10.1, Y1.1
- net N$40: now also IC3.42, R13.1; no longer IC4.42, R24.1
- net N$41: now also R2.1; no longer R26.1
- net N$42: now also Q1.3; no longer Q2.3
- net N$5: now also IC3.1; no longer IC4.1
- net N$6: now also R10.2; no longer R1.2
- net N$7: now also S4.2; no longer S3.2
- net N$8: now also LED2.K, Q2.3; no longer LED1.K, Q1.3
- net SWDCLK: now also IC3.37; no longer IC4.37
- net SWDIO: now also IC3.34; no longer IC4.34
- net USART_RX: now also R7.1; no longer R23.1
- net USART_TX: now also R6.1; no longer R22.1
- net VOUT: now also IC4.2; no longer IC5.2
Other:
- board size 80 x 40 mm -> 90 x 50 mm

Commit message: wiring
Parts:
- added JP_LED_MCU, JP_LED_TM1809: (no value), SparkFun-Connectors:1X03
- moved C2 63.0 mm to (88.0, 26.0)
- moved C3 63.0 mm to (88.0, 23.0)
- moved IC2 63.0 mm to (87.0, 12.0)
- moved LED1 63.0 mm to (82.0, 21.0)
- moved LED3 63.0 mm to (92.0, 21.0)
- moved LED4 63.0 mm to (92.0, 19.0)
- moved LED5 63.0 mm to (92.0, 17.0)
- moved LED6 63.0 mm to (92.0, 15.0)
- moved LED7 63.0 mm to (92.0, 13.0)
- moved LED8 63.0 mm to (92.0, 11.0)
- moved R16 63.0 mm to (96.0, 21.0)
- moved R19 63.0 mm to (96.0, 19.0)
- moved R20 63.0 mm to (96.0, 17.0)
- moved R21 63.0 mm to (96.0, 15.0)
- moved R22 63.0 mm to (96.0, 13.0)
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Connections:
- removed net LED_CTRL: IC2.14, R12.1
- removed net VOUT: C15.1, C16.1, IC4.2
- new net LED_MCU: JP_LED_MCU.3
- new net LED_TM: IC2.14, JP_LED_TM1809.3, R12.1
- net 3.3V: now also C15.1, C16.1, C4.1, IC4.2
- net 5V: now also JP_LED_MCU.1, JP_LED_TM1809.1; no longer C4.1
- net GND: now also JP_LED_MCU.2, JP_LED_TM1809.2
Routing:
- net N$20: track 0.00 -> 29.1 mm
- net GND: track 0.00 -> 18.7 mm
- net 5V: track 0.00 -> 14.8 mm, vias 0 -> 1
- net N$10: track 0.00 -> 14.1 mm, vias 0 -> 2
- net N$7: track 0.00 -> 12.4 mm
- net N$22: track 0.00 -> 9.72 mm
- net N$25: track 0.00 -> 5.02 mm, vias 0 -> 1
- net N$23: track 0.00 -> 2.37 mm
- added copper zone on layer 1, net GND
- added copper zone on layer 16, net GND
Other:
- board size 90 x 50 mm -> 113 x 50 mm

Commit message: wiring
Parts:
- moved R15 41.2 mm to (16.0, 20.5), turned to 270 degrees
- moved C10 35.8 mm to (37.0, 45.5)
- moved C11 35.8 mm to (37.0, 43.5)
- moved R25 34.3 mm to (24.0, 28.5)
- moved C15 33.3 mm to (37.0, 36.5), turned to 180 degrees
- moved C16 33.3 mm to (37.0, 34.5), turned to 180 degrees
- moved Y1 30.6 mm to (23.5, 32.0), turned to 180 degrees
- moved S3 30.3 mm to (39.0, 15.5)
- moved IC4 29.2 mm to (37.0, 40.0)
- moved R24 28.2 mm to (26.5, 11.0), turned to 90 degrees
- moved C14 26.4 mm to (22.0, 36.0), flipped to the bottom, turned to 90 degrees
- moved C13 25.8 mm to (25.0, 36.0), flipped to the bottom, turned to 90 degrees
- moved R14 25.3 mm to (46.5, 22.5), flipped to the bottom, turned to 0 degrees
- moved R1 19.9 mm to (30.0, 33.5), flipped to the bottom, turned to 0 degrees
- moved R13 19.4 mm to (46.5, 25.0), flipped to the bottom
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Routing:
- net 5V: track 14.8 -> 136.9 mm, vias 1 -> 2
- net N$8: track 0.00 -> 17.7 mm
- net N$3: track 0.00 -> 17.5 mm
- net N$14: track 0.00 -> 14.8 mm
- net GND: track 18.7 -> 32.2 mm
- net N$4: track 0.00 -> 13.0 mm
- net N$12: track 0.00 -> 11.9 mm
- net N$11: track 0.00 -> 10.7 mm
- net N$37: track 0.00 -> 6.58 mm
- net N$38: track 0.00 -> 5.75 mm
- net 3.3V: track 0.00 -> 4.62 mm
- net N$5: track 0.00 -> 4.44 mm
- net USART_RX: track 0.00 -> 4.17 mm
- net USART_TX: track 0.00 -> 4.15 mm
- net N$9: track 0.00 -> 2.95 mm
Other:
- board size 113 x 50 mm -> 113 x 46.5 mm

Commit message: nearly finish
Parts:
- added R28: 10K, SparkFun-Passives:0603-RES
- moved R12 53.9 mm to (82.5, 2.50), turned to 270 degrees
- moved R9 45.1 mm to (76.5, 18.5), turned to 90 degrees
- moved C12 42.7 mm to (18.5, 29.5), turned to 180 degrees
- moved R16 28.3 mm to (75.5, 1.50), turned to 180 degrees
- moved JP_LED_TM1809 27.1 mm to (76.5, 22.5)
- moved C2 25.7 mm to (77.5, 2.50), flipped to the bottom, turned to 90 degrees
- moved R19 25.7 mm to (75.5, 3.50), turned to 180 degrees
- moved R20 23.5 mm to (75.5, 5.50), turned to 180 degrees
- moved LED3 22.1 mm to (81.5, 1.50), turned to 270 degrees
- moved C3 22.0 mm to (80.0, 2.50), flipped to the bottom, turned to 90 degrees
- moved R21 21.8 mm to (75.5, 7.50), turned to 180 degrees
- moved R22 20.8 mm to (75.5, 9.50), turned to 180 degrees
- moved R23 20.5 mm to (75.5, 11.5), turned to 180 degrees
- moved LED4 18.7 mm to (81.5, 3.50), turned to 270 degrees
- moved LED5 15.6 mm to (81.5, 5.50), turned to 270 degrees
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Connections:
- new net N$44: C12.1, IC3.7, R28.1
- net 3.3V: now also R28.2; no longer C12.1, IC3.7
- net 5V: no longer C2.1, C3.1, R12.2
- net BTN_RELOAD: now also IC3.46
- net BTN_TRIGGER: now also IC3.41
- net BUZZER: now also IC3.12
- net DIP_SW1: now also IC3.27
- net DIP_SW2: now also IC3.26
- net DIP_SW3: now also IC3.25
- net GND: now also C2.1, C3.1, JP_LED_MCU.3, JP_LED_TM1809.3; no longer C2.2, C3.2, JP_LED_MCU.2, JP_LED_TM1809.2
- net IR_EMITTER: now also IC3.15
- net IR_RECEIVE1: now also IC3.21
- net IR_RECEIVE2: now also IC3.22
- net LED_MCU: now also IC3.45, JP_LED_MCU.2; no longer JP_LED_MCU.3
- net LED_TM: now also JP_LED_TM1809.2; no longer JP_LED_TM1809.3
- net N$36: now also C2.2, C3.2, R12.2
- net PWM_38K: now also IC3.16
Routing:
- net 3.3V: track 4.62 -> 95.8 mm, vias 0 -> 5
- net 5V: track 136.9 -> 203.8 mm, vias 2 -> 5
- net BTN_RELOAD: track 0.00 -> 37.3 mm
- net BTN_TRIGGER: track 0.00 -> 36.3 mm
- net IR_RECEIVE1: track 0.00 -> 31.7 mm, vias 0 -> 1
- net N$2: track 0.00 -> 28.7 mm, vias 0 -> 1
- net N$36: track 0.00 -> 27.1 mm
- net LED_TM: track 0.00 -> 21.4 mm, vias 0 -> 1
- net DIP_SW3: track 0.00 -> 20.3 mm, vias 0 -> 1
- net N$39: track 0.00 -> 20.2 mm, vias 0 -> 1
- net N$40: track 0.00 -> 18.4 mm, vias 0 -> 1
- net N$16: track 0.00 -> 17.8 mm, vias 0 -> 1
- net DIP_SW2: track 0.00 -> 16.9 mm, vias 0 -> 1
- net SWDCLK: track 0.00 -> 15.8 mm
- net IR_RECEIVE2: track 0.00 -> 15.5 mm
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Other:
- board size 113 x 46.5 mm -> 86.5 x 46.5 mm

Commit message: finish wire
Parts:
- added Q3, Q4: 2N7002, SparkFun-DiscreteSemi:SOT23
- added R29, R30: 47K, SparkFun-Passives:0603-RES
- added R31, R32: 10K, SparkFun-Passives:0603-RES
- R13, R14: value 220R -> 100R
- R17: value 110K -> 110K(47K)
- R18: value 15K -> 15K(6.4K)
- moved C2 22.0 mm to (76.5, 24.5)
- moved C3 22.0 mm to (79.0, 24.5)
- moved IC2 22.0 mm to (79.0, 32.0)
- moved LED1 22.0 mm to (81.0, 38.5)
- moved LED3 22.0 mm to (80.5, 23.5)
- moved LED4 22.0 mm to (80.5, 25.5)
- moved LED5 22.0 mm to (80.5, 27.5)
- moved LED6 22.0 mm to (80.5, 29.5)
- moved LED7 22.0 mm to (80.5, 31.5)
- moved LED8 22.0 mm to (80.5, 33.5)
- moved R12 22.0 mm to (81.5, 24.5)
- moved R9 22.0 mm to (75.5, 40.5)
- moved JP_LED_TM1809 22.0 mm to (77.0, 44.5)
- moved R16 22.0 mm to (75.0, 23.5)
- moved R19 22.0 mm to (75.0, 25.5)
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Connections:
- new net N$45: IC5.1, Q3.3, R30.1
- new net N$47: IC6.1, Q4.3, R29.1
- net 3.3V: now also Q3.1, Q4.1, R31.2, R32.2
- net 5V: now also R29.2, R30.2
- net IR_EMITTER: now also IC3.21; no longer IC3.15
- net IR_RECEIVE1: now also IC3.13, Q3.2, R31.1; no longer IC3.21, IC5.1
- net IR_RECEIVE2: now also Q4.2, R32.1; no longer IC6.1
Routing:
- net GND: track 32.2 -> 514.7 mm, vias 0 -> 76
- net 3.3V: track 95.8 -> 110.8 mm, vias 5 -> 6
- net IR_RECEIVE1: track 31.7 -> 18.0 mm
- net N$45: track 0.00 -> 6.55 mm
- net IR_RECEIVE2: track 15.5 -> 9.10 mm
- net N$47: track 0.00 -> 6.32 mm
- net IR_EMITTER: track 9.75 -> 14.3 mm
- net N$11: track 10.7 -> 14.7 mm
- net N$39: track 20.2 -> 17.5 mm
- net BTN_RELOAD: track 37.3 -> 35.2 mm, vias 0 -> 2
- net N$6: track 5.84 -> 4.14 mm
- net 5V: track 203.8 -> 205.4 mm
- net N$12: track 11.9 -> 13.3 mm
- net PWM_38K: track 10.6 -> 9.47 mm
- net USART_TX: track 4.15 -> 3.15 mm
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Other:
- board size 86.5 x 46.5 mm -> 85.5 x 45 mm

Commit message: finish
Parts:
- removed IR_LASER, JP_LED_MCU, JP_LED_TM1809: (no value), SparkFun-Connectors:1X03
- removed JP1: M02PTH, SparkFun-Connectors:1X02
- removed L3: 4.7uh, SparkFun-Passives:CR75_V2
- removed S4: (no value), digital-toy:SWITCH-SPDT-AM#6
- removed U$1: RJ9PTH, SparkFun-Connectors:RJ9
- added J1: RJ9PTH, SparkFun-Connectors:RJ9
- added JP2, JP4, LED: (no value), SparkFun-Connectors:1X03
- added JP3: M02PTH, SparkFun-Connectors:1X02
- added L1: 4.7uh, SparkFun-Passives:CR75_V2
- added POWER: (no value), digital-toy:SWITCH-SPDT-AM#6
- added R33, R34: 10K, SparkFun-Passives:0603-RES
- C22: device SparkFun-Passives:0402-CAP -> SparkFun-Passives:0603-CAP
- C24: device SparkFun-Passives:0603-CAP -> SparkFun-Passives:0402-CAP
- C3: value 1uf -> 100nf; device SparkFun-Passives:0603-CAP -> SparkFun-Passives:0402-CAP
- C4: value 100nf -> 10uf; device SparkFun-Passives:0603-CAP -> SparkFun-Passives:0402-CAP
- C5: value 100nf -> 1uf; device SparkFun-Passives:0402-CAP -> SparkFun-Passives:0603-CAP
- C6: value 10uf -> 100nf; device SparkFun-Passives:0402-CAP -> SparkFun-Passives:0603-CAP
- R25: value 1m -> 10K
- R26: value 100R -> 1m
- R28: value 10K -> 100R
- moved C2 62.0 mm to (14.5, 26.0), turned to 180 degrees
- moved C4 42.1 mm to (56.5, 31.0), flipped to the top
- moved R30 34.8 mm to (15.5, 7.50), turned to 0 degrees
- moved R29 32.2 mm to (12.0, 37.5), flipped to the top, turned to 180 degrees
- moved Q3 31.5 mm to (16.5, 7.50), flipped to the top, turned to 180 degrees
- moved R27 28.6 mm to (7.50, 37.5), flipped to the bottom, turned to 0 degrees
- moved Q4 28.5 mm to (17.0, 37.5), flipped to the bottom, turned to 0 degrees
- moved R24 26.9 mm to (18.5, 25.5), flipped to the top
- moved R25 25.7 mm to (38.0, 5.50), flipped to the bottom, turned to 180 degrees
- moved C5 23.7 mm to (79.0, 23.0), flipped to the bottom, turned to 90 degrees
- moved R31 23.0 mm to (16.5, 11.5), flipped to the top, turned to 0 degrees
- moved C23 23.0 mm to (12.0, 11.5), flipped to the top, turned to 0 degrees
- moved C3 22.9 mm to (56.5, 29.0), flipped to the top, turned to 180 degrees
- moved R28 22.4 mm to (7.57, 7.45)
- moved C6 22.1 mm to (76.5, 23.0), flipped to the bottom, turned to 90 degrees
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Connections:
- net BTN_TRIGGER renamed BTN_F1
- net 3.3V: now also C2.1, C24.1, R24.2; no longer C22.1, C4.1, R28.2
- net 5V: now also J1.1, JP2.1, LED.1, R28.2, R33.2, R34.2; no longer JP_LED_MCU.1, JP_LED_TM1809.1, R26.2, R29.2, R30.2, U$1.1
- net GND: now also C2.2, C3.2, C5.1, C6.1, J1.4, JP2.3, JP3.1, JP4.3, LED.3, R25.1; no longer C2.1, C3.1, C5.2, C6.2, IR_LASER.3, JP1.1, JP_LED_MCU.3, JP_LED_TM1809.3, R24.1, U$1.4
- net I2C_SCL: now also J1.2, R34.1; no longer U$1.2
- net I2C_SDA: now also J1.3, R33.1; no longer U$1.3
- net IR_RECEIVE1: now also Q4.2, R32.1; no longer Q3.2, R31.1
- net IR_RECEIVE2: now also Q3.2, R31.1; no longer Q4.2, R32.1
- net LED_MCU: now also LED.2; no longer JP_LED_MCU.2
- net LED_TM: now also JP2.2; no longer JP_LED_TM1809.2
- net N$10: now also POWER.3; no longer S4.3
- net N$11: now also C22.1, R27.1, R29.2; no longer C23.1, R26.1
- net N$12: now also C23.1, R28.1, R30.2; no longer C24.1, R27.1
- net N$14: now also JP4.1; no longer IR_LASER.1
- net N$2: now also R25.2; no longer R24.2
- net N$20: now also C3.1, C4.1, L1.P$1; no longer C5.1, C6.1, L3.P$1
- net N$22: now also L1.P$2; no longer L3.P$2
- net N$3: now also R26.2; no longer R25.2
- net N$36: now also C5.2, C6.2; no longer C2.2, C3.2
- net N$4: now also R26.1; no longer R25.1
- net N$44: now also R24.1; no longer R28.1
- net N$45: now also Q4.3, R29.1; no longer Q3.3, R30.1
- net N$47: now also Q3.3, R30.1; no longer Q4.3, R29.1
- net N$7: now also JP3.2, POWER.2; no longer JP1.2, S4.2
- net N$8: now also JP4.2; no longer IR_LASER.2
Routing:
- net 5V: track 205.4 -> 191.2 mm, vias 5 -> 3
- net GND: track 514.7 -> 505.2 mm
- net N$12: track 13.3 -> 18.7 mm
- net I2C_SDA: track 7.59 -> 12.1 mm
- net I2C_SCL: track 6.49 -> 10.3 mm
- net N$11: track 14.7 -> 18.3 mm
- net N$45: track 6.55 -> 8.62 mm
- net N$47: track 6.32 -> 7.22 mm
- net USART_TX: track 3.15 -> 3.65 mm
- net USART_RX: track 3.17 -> 3.67 mm
- net N$38: track 5.75 -> 5.25 mm
- net N$37: track 6.58 -> 6.08 mm
Other:
- outline, holes or cut-outs redrawn
- board text added: "C"
- board text added: "C1"
- board text added: "FIRE"
- board text added: "Function"
- board text added: "G"
- board text added: "IO"
- board text added: "R"
- board text added: "T"
- board text added: "V"

Commit message: found some mistake, wait fixup
Parts:
- removed C3, C9: 100nf, SparkFun-Passives:0402-CAP
- removed C4, C7, C8: 10uf, SparkFun-Passives:0402-CAP
- added C25, C29: 100nf, SparkFun-Passives:0603-CAP
- added C26, C27, C28: 10uf, SparkFun-Passives:0603-CAP
Connections:
- net 5V: now also C27.2, C28.2, C29.2; no longer C7.1, C8.1, C9.1
- net GND: now also C25.2, C26.2, C27.1, C28.1, C29.1; no longer C3.2, C4.2, C7.2, C8.2, C9.2
- net N$20: now also C25.1, C26.1; no longer C3.1, C4.1
Routing:
- net GND: track 505.2 -> 496.5 mm
- net 5V: track 191.2 -> 187.0 mm
- net N$20: track 29.1 -> 29.8 mm

Commit message: modify some packages
Parts:
- removed C16, C17, C18, C21: 100nf, SparkFun-Passives:0402-CAP
- removed C24: 4.7uf, SparkFun-Passives:0402-CAP
- removed U1: 74LVC1G08SE-7, SparkFun-DigitalIC:SOT353
- added C3, C7: 1uf, SparkFun-Passives:0603-CAP
- added C4, C8, C9: 100nf, SparkFun-Passives:0603-CAP
- added U$1: SN74LVC1G08, SparkFun-DigitalIC:SOT23-5
- C10: value 1uf -> 100nf; device SparkFun-Passives:0402-CAP -> SparkFun-Passives:0603-CAP
- C11: device SparkFun-Passives:0402-CAP -> SparkFun-Passives:0603-CAP
- C15: value 1uf -> 4.7uf; device SparkFun-Passives:0402-CAP -> SparkFun-Passives:0603-CAP
- moved C10 29.8 mm to (23.5, 13.5), flipped to the bottom, turned to 270 degrees
- moved C11 23.3 mm to (27.0, 17.0), flipped to the bottom
- moved C15 16.7 mm to (23.5, 20.5), flipped to the bottom, turned to 90 degrees
- moved R34 10.3 mm to (44.0, 16.0), flipped to the bottom, turned to 90 degrees
- moved R33 4.61 mm to (44.0, 19.5), flipped to the bottom, turned to 270 degrees
- moved C27 3.16 mm to (47.5, 31.0)
- moved C28 3.04 mm to (45.5, 31.0)
- moved C29 3.04 mm to (43.5, 31.0)
- moved R14 1.58 mm to (46.5, 19.5), turned to 90 degrees
- moved R13 0.71 mm to (46.5, 16.0), turned to 270 degrees
- moved C2 0.50 mm to (14.5, 25.5)
- moved IC4 0.50 mm to (36.0, 35.5)
- moved R17 0.50 mm to (48.0, 33.0)
Connections:
- net 3.3V: now also C10.1, C11.1, C7.1, C8.1, C9.1, U$1.5; no longer C16.1, C17.1, C18.1, C21.1, C24.1, U1.5
- net 5V: now also C3.1, C4.1; no longer C10.1, C11.1
- net GND: now also C3.2, C4.2, C7.2, C8.2, C9.2, U$1.3; no longer C16.2, C17.2, C18.2, C21.2, C24.2, U1.3
- net I2C_SCL: now also IC3.42; no longer J1.2
- net I2C_SDA: now also IC3.43; no longer J1.3
- net IR_EMITTER: now also U$1.1; no longer U1.1
- net N$39: now also J1.3; no longer IC3.43
- net N$40: now also J1.2; no longer IC3.42
- net N$6: now also U$1.4; no longer U1.4
- net PWM_38K: now also U$1.2; no longer U1.2
Routing:
- net N$40: track 17.7 -> 6.42 mm, vias 1 -> 0
- net I2C_SCL: track 10.3 -> 19.2 mm, vias 0 -> 1
- net I2C_SDA: track 12.1 -> 19.8 mm
- net GND: track 496.5 -> 503.9 mm
- net N$39: track 17.5 -> 11.4 mm, vias 1 -> 0
- net 5V: track 187.0 -> 188.8 mm, vias 3 -> 4
- net BTN_RELOAD: track 35.2 -> 36.9 mm
- net 3.3V: track 110.8 -> 112.3 mm
- net N$6: track 4.14 -> 2.87 mm
- net PWM_38K: track 9.47 -> 8.32 mm
- net IR_EMITTER: track 14.3 -> 13.5 mm
- net N$25: track 5.02 -> 5.52 mm
