File: hardware/v0.1/1.brd (EAGLE design)
At the start: 85.5 x 45 mm, 95 parts, among them IC1 FP6291, IC2 TM1809, IC3 STM32F10XCXT6, IC5 TSOP34830, IC6 TSOP34830, J1 RJ9PTH, Q1 8050, Q2 8050, Q3 2N7002, Q4 2N7002, Y1 8M

Commit message: update silkscreen
Parts:
- removed C25, C29: 100nf, SparkFun-Passives:0603-CAP
- removed C26, C27, C28: 10uf, SparkFun-Passives:0603-CAP
- removed U$1: SN74LVC1G08, SparkFun-DigitalIC:SOT23-5
- added C16, C17, C18, C21: 100nf, SparkFun-Passives:0603-CAP
- added C24: 4.7uf, SparkFun-Passives:0603-CAP
- added IC7: TSOP34830, vishay-1:TSOP348
- C10: value 100nf -> 1uf
- C15: value 4.7uf -> 1uf
- C3: value 1uf -> 100nf
- C4, C8: value 100nf -> 10uf
- C7: value 1uf -> 10uf
- IC1: value FP6291 -> SN74LVC1G08; device eagle_lib_lishen:SOT23-6 -> SparkFun-DigitalIC:SOT23-5
- IC2: value TM1809 -> FP6291; device eagle_lib_lishen:SOP-14 -> eagle_lib_lishen:SOT23-6
- IC3: value STM32F10XCXT6 -> TM1809; device stm32:TQFP48 -> eagle_lib_lishen:SOP-14
- IC4: value (none) -> STM32F10XCXT6; device SparkFun-PowerIC:SOT23-3 -> stm32:TQFP48
- IC5: value TSOP34830 -> (none); device vishay-1:TSOP348 -> SparkFun-PowerIC:SOT23-3
- R10: value 2.2K -> 220R
- R11: value 51 -> 220R; device SparkFun-Resistors:1206 -> SparkFun-Passives:0603-RES
- R12: value 10K -> 47k
- R14: value 100R -> 2.2K
- R15: value 10K -> 51; device SparkFun-Passives:0603-RES -> SparkFun-Resistors:1206
- R16, R5: value 470R -> 10K
- R17: value 110K(47K) -> 10K
- R18: value 15K(6.4K) -> 470R
- R19: value 470R -> 110K(47K)
- R20: value 470R -> 15K(6.4K)
- R24, R25: value 10K -> 470R
- R26: value 1m -> 10K
- R27: value 100R -> 10K
- R28: value 100R -> 1m
- R29, R30: value 47K -> 100R
- R3, R4: value 470R -> 100R
- R31, R32: value 10K -> 47K
- R6: value 220R -> 10K
- R7: value 220R -> 470R
- R8: value 47k -> 470R
- R9: value 100R -> 470R
- moved R7 58.9 mm to (75.0, 35.0), turned to 180 degrees
- moved IC3 57.1 mm to (79.0, 30.5), flipped to the bottom, turned to 90 degrees
- moved R24 56.7 mm to (75.0, 30.0)
- moved R25 45.5 mm to (75.0, 32.0), flipped to the top
- moved R27 44.2 mm to (38.0, 5.50), turned to 180 degrees
- moved IC1 41.9 mm to (14.5, 21.5), flipped to the bottom
- moved R17 39.8 mm to (12.0, 16.0), flipped to the top, turned to 180 degrees
- moved IC6 38.0 mm to (13.5, 41.5), flipped to the top, turned to 180 degrees
- moved R13 37.0 mm to (75.5, 39.0), turned to 90 degrees
- moved R4 36.6 mm to (46.5, 16.0), flipped to the bottom, turned to 270 degrees
- moved R14 36.0 mm to (10.5, 21.0), flipped to the top, turned to 270 degrees
- moved R5 35.6 mm to (44.0, 19.5), flipped to the bottom, turned to 270 degrees
- moved R3 32.4 mm to (46.5, 19.5), flipped to the bottom, turned to 90 degrees
- moved R34 31.9 mm to (17.0, 33.0), turned to 180 degrees
- moved C10 31.1 mm to (36.0, 42.0), flipped to the top, turned to 180 degrees
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- renumbered LED to JP1, POWER to S4, SWD to JP7, UPDATE to JP5, USART to JP6
Connections:
- net 3.3V: now also C16.1, C17.1, C18.1, C21.1, C24.1, IC1.5, IC4.24, IC4.36, IC4.48, IC4.9, IC5.2, R26.2, R33.2, R34.2; no longer C10.1, C11.1, C7.1, C8.1, C9.1, IC3.24, IC3.36, IC3.48, IC3.9, IC4.2, R24.2, R31.2, R32.2, U$1.5
- net 5V: now also C10.1, C11.1, C7.2, C8.2, C9.2, IC5.3, R13.2, R15.2, R18.2, R24.2, R25.2, R29.2, R30.2, R6.2, R7.2, R8.2; no longer C27.2, C28.2, C29.2, C3.1, C4.1, IC4.3, R11.2, R16.2, R17.2, R20.2, R27.2, R28.2, R3.2, R33.2, R34.2, R4.2
- net BTN_F1: now also IC4.41; no longer IC3.41
- net BTN_RELOAD: now also IC4.46; no longer IC3.46
- net BUZZER: now also IC4.12; no longer IC3.12
- net DIP_SW1: now also IC4.27; no longer IC3.27
- net DIP_SW2: now also IC4.26; no longer IC3.26
- net DIP_SW3: now also IC4.25; no longer IC3.25
- net GND: now also C16.2, C17.2, C18.2, C21.2, C24.2, C7.1, C8.1, C9.1, IC1.3, IC2.2, IC3.7, IC4.23, IC4.35, IC4.47, IC4.8, IC5.1, IC7.2, R12.1, R17.2, R20.1, R27.1; no longer C25.2, C26.2, C27.1, C28.1, C29.1, C7.2, C8.2, C9.2, IC1.2, IC2.7, IC3.23, IC3.35, IC3.47, IC3.8, IC4.1, IC5.2, R15.2, R18.1, R25.1, R8.1, U$1.3
- net I2C_SCL: now also IC4.42, R4.2, R6.1; no longer IC3.42, R13.2, R34.1
- net I2C_SDA: now also IC4.43, R3.2, R5.1; no longer IC3.43, R14.2, R33.1
- net IR_EMITTER: now also IC1.1, IC4.21; no longer IC3.21, U$1.1
- net IR_RECEIVE1: now also IC4.13, R34.1; no longer IC3.13, R32.1
- net IR_RECEIVE2: now also IC4.22, R33.1; no longer IC3.22, R31.1
- net LED_MCU: now also IC4.45; no longer IC3.45
- net LED_TM: now also IC3.14, R16.1; no longer IC2.14, R12.1
- net N$1: now also IC4.20, R17.1; no longer IC3.20, R15.1
- net N$11: now also IC6.3, R29.1, R31.2; no longer IC5.3, R27.1, R29.2
- net N$12: now also IC7.3, R30.1, R32.2; no longer IC6.3, R28.1, R30.2
- net N$13: now also IC3.4; no longer IC2.4
- net N$14: now also R15.1; no longer R11.1
- net N$15: now also IC3.5; no longer IC2.5
- net N$16: now also IC3.6; no longer IC2.6
- net N$17: now also R9.1; no longer R5.1
- net N$18: now also R8.1; no longer R4.1
- net N$19: now also R7.1; no longer R3.1
- net N$2: now also IC4.44, R27.2; no longer IC3.44, R25.2
- net N$20: now also C3.1, C4.1, IC2.4, IC2.5; no longer C25.1, C26.1, IC1.4, IC1.5
- net N$21: now also IC3.13; no longer IC2.13
- net N$22: now also IC2.1; no longer IC1.1
- net N$23: now also IC2.6, R12.2; no longer IC1.6, R8.2
- net N$24: now also R18.1; no longer R16.1
- net N$25: now also IC2.3, R19.1, R20.2; no longer IC1.3, R17.1, R18.2
- net N$26: now also R21.1; no longer R19.1
- net N$27: now also IC3.12; no longer IC2.12
- net N$28: now also IC3.11; no longer IC2.11
- net N$29: now also IC3.10; no longer IC2.10
- net N$3: now also IC4.5, R28.2; no longer IC3.5, R26.2
- net N$30: now also IC3.9; no longer IC2.9
- net N$31: now also IC3.8; no longer IC2.8
- net N$32: now also R22.1; no longer R20.1
- net N$33: now also R23.1; no longer R21.1
- net N$34: now also R24.1; no longer R22.1
- net N$35: now also R25.1; no longer R23.1
- net N$36: now also IC3.1, R13.1, R16.2; no longer IC2.1, R12.2, R9.1
- net N$37: now also IC4.30, R10.2; no longer IC3.30, R6.2
- net N$38: now also IC4.31, R11.2; no longer IC3.31, R7.2
- net N$39: now also R3.1; no longer R14.1
- net N$4: now also IC4.6, R28.1; no longer IC3.6, R26.1
- net N$40: now also R4.1; no longer R13.1
- net N$44: now also IC4.7, R26.1; no longer IC3.7, R24.1
- net N$45: now also IC6.1, R31.1; no longer IC5.1, R29.1
- net N$47: now also IC7.1, R32.1; no longer IC6.1, R30.1
- net N$5: now also IC4.1; no longer IC3.1
- net N$6: now also IC1.4, R14.2; no longer R10.2, U$1.4
- net N$9: now also R14.1; no longer R10.1
- net PWM_38K: now also IC1.2, IC4.16; no longer IC3.16, U$1.2
- net SWDCLK: now also IC4.37; no longer IC3.37
- net SWDIO: now also IC4.34; no longer IC3.34
- net USART_RX: now also R11.1; no longer R7.1
- net USART_TX: now also R10.1; no longer R6.1
