File: hardware/v0.1/1.sch (EAGLE design)
At the start: 84 parts, among them IC1 FP6291, IC2 TSOP34830, IC3 TSOP34830, IC4 STM32F10XCXT6, IC6 TM1809, Q1 8050, Q2 8050, U1 74LVC1G08SE-7, Y1 8m

Commit message: start wiring
Parts:
- removed L1: 4.7uh, SparkFun-Passives:INDUCTORIHLP4040DZ
- added L3: 4.7uh, SparkFun-Passives:INDUCTORCR75_V2
- C1: value 100nf -> 100uf; device SparkFun-Passives:CAP0402-CAP -> SparkFun-Capacitors:CAP_POL6032
- C10: value 4.7uf -> 1uf; device SparkFun-Passives:CAP0603-CAP -> SparkFun-Passives:CAP0402-CAP
- C19: device SparkFun-Passives:CAP0402-CAP -> SparkFun-Passives:CAP0603-CAP
- C2, C4: value 10uf -> 100nf; device SparkFun-Passives:CAP0402-CAP -> SparkFun-Passives:CAP0603-CAP
- C20: value 4.7uf -> 100nf; device SparkFun-Passives:CAP0402-CAP -> SparkFun-Passives:CAP0603-CAP
- C21: value 100uf -> 100nf; device SparkFun-Capacitors:CAP_POL6032 -> SparkFun-Passives:CAP0402-CAP
- C22: value 100nf -> 4.7uf; device SparkFun-Passives:CAP0603-CAP -> SparkFun-Passives:CAP0402-CAP
- C23: value 1uf -> 4.7uf
- C24: value 100nf -> 4.7uf
- C3: value 10uf -> 1uf; device SparkFun-Passives:CAP0402-CAP -> SparkFun-Passives:CAP0603-CAP
- C6, C7: value 100nf -> 10uf; device SparkFun-Passives:CAP0603-CAP -> SparkFun-Passives:CAP0402-CAP
- C8: value 1uf -> 10uf
- C9: value 4.7uf -> 100nf; device SparkFun-Passives:CAP0603-CAP -> SparkFun-Passives:CAP0402-CAP
- D1: device SparkFun-DiscreteSemi:DIODE-SCHOTTKT-SMB -> SparkFun-DiscreteSemi:DIODE-SCHOTTKY_
- IC2: value TSOP34830 -> TM1809; device vishay-1:TSOP34830 -> eagle_lib_lishen:TM1809
- IC3: value TSOP34830 -> STM32F10XCXT6; device vishay-1:TSOP34830 -> stm32:STM32F10XCXT6
- IC4: value STM32F10XCXT6 -> (none); device stm32:STM32F10XCXT6 -> SparkFun-PowerIC:XC6206
- IC5: value (none) -> TSOP34830; device SparkFun-PowerIC:XC6206 -> vishay-1:TSOP34830
- IC6: value TM1809 -> TSOP34830; device eagle_lib_lishen:TM1809 -> vishay-1:TSOP34830
- LED1: value IR -> LED-TRICOLOR-5050NO_IC; device SparkFun-LED:LED5MM -> SparkFun-LED:LED-TRICOLOR-5050NO_IC
- LED2: value LED-TRICOLOR-5050NO_IC -> IR; device SparkFun-LED:LED-TRICOLOR-5050NO_IC -> SparkFun-LED:LED5MM
- R10: value 1m -> 2.2K
- R11: value 470R -> 51; device SparkFun-Passives:RESISTOR0603-RES -> SparkFun-Resistors:RESISTOR1206
- R12, R15: value 470R -> 10K
- R13, R14: value 470R -> 220R
- R17: value 470R -> 110K
- R18: value 470R -> 15K
- R2: value 51R -> 180R
- R20: value 100R -> 470R
- R21, R4: value 10K -> 470R
- R22, R23: value 220R -> 470R
- R24: value 220R -> 10K
- R25: value 220R -> 1m
- R26: value 180R -> 100R
- R27: value 2.2K -> 100R
- R3: value 47k -> 470R
- R5: value 110K -> 470R
- R6: value 15K -> 220R
- R7: value 100R -> 220R
- R8: value 100R -> 47k
- R9: value 10K -> 100R
- S3: device digital-toy:SWITCH-SPST3AM6 -> switch-dil:DIP03YL
- S4: device switch-dil:DIP03YL -> digital-toy:SWITCH-SPST3AM6
- Y1: value 8m -> 8M; device SparkFun-FreqCtrl:CRYSTALHC49US -> SparkFun-FreqCtrl:CRYSTALTXC-7A
Connections:
- removed net N$43 (its old number): Q2.B, R27.1
- new net N$9: Q2.B, R10.1
- net 3.3V: now also C21.1, C22.1, IC3AN_POWER.VDDA, IC3POWER.VDD_1, IC3POWER.VDD_2, IC3POWER.VDD_3, IC3RESET.NRST; no longer C19.1, C20.1, IC4AN_POWER.VDDA, IC4POWER.VDD_1, IC4POWER.VDD_2, IC4POWER.VDD_3, IC4RESET.NRST
- net 5V: now also C1.+, C10.1, C2.1, C7.1, C9.1, IC4.VIN, R22.2, R23.2, R27.2, R3.2, R4.2, R9.2; no longer C21.+, C22.1, C23.1, C24.1, C5.1, IC5.VIN, R13.2, R14.2, R15.2, R18.2, R7.2, R8.2
- net BUZZER: now also R1.2; no longer R27.2
- net DIP_SW1: now also S3.1; no longer S4.1
- net DIP_SW2: now also S3.2; no longer S4.2
- net DIP_SW3: now also S3.3; no longer S4.3
- net GND: now also C1.-, C21.2, IC3AN_POWER.VSSA, IC3POWER.VSS_1, IC3POWER.VSS_2, IC3POWER.VSS_3, IC4.VSS, IC5.GND, R15.2, R18.1, R24.1, R8.1, S3.4, S3.5, S3.6; no longer C1.2, C21.-, IC3.GND, IC4AN_POWER.VSSA, IC4POWER.VSS_1, IC4POWER.VSS_2, IC4POWER.VSS_3, IC5.VSS, R3.1, R4.2, R6.1, R9.1, S4.4, S4.5, S4.6
- net I2C_SCL: now also R13.2; no longer R24.2
- net I2C_SDA: now also R14.2; no longer R25.2
- net IR_RECEIVE1: now also IC5.OUT; no longer IC2.OUT
- net IR_RECEIVE2: now also IC6.OUT; no longer IC3.OUT
- net LED_CTRL: now also IC2.DIN, R12.1; no longer IC6.DIN, R21.1
- net N$1: now also IC3PORTB_L.PB2, R15.1; no longer IC4PORTB_L.PB2, R4.1
- net N$10: now also S4.S; no longer S3.S
- net N$11: now also C19.1, C23.1, IC5.VS, R26.1; no longer C6.1, C9.1, IC2.VS, R7.1
- net N$12: now also C20.1, C24.1, IC6.VS, R27.1; no longer C10.1, C7.1, IC3.VS, R8.1
- net N$13: now also IC2.3OUTR, LED1.RED-C; no longer IC6.3OUTR, LED2.RED-C
- net N$14: now also LED2.A, R11.1; no longer LED1.A, R2.1
- net N$15: now also IC2.3OUTG, LED1.GRN-C; no longer IC6.3OUTG, LED2.GRN-C
- net N$16: now also IC2.3OUTB, LED1.BLU-C; no longer IC6.3OUTB, LED2.BLU-C
- net N$17: now also LED1.RED-A, R5.1; no longer LED2.RED-A, R11.1
- net N$18: now also LED1.GRN-A, R4.1; no longer LED2.GRN-A, R12.1
- net N$19: now also LED1.BLU-A, R3.1; no longer LED2.BLU-A, R13.1
- net N$2: now also IC3RESET.BOOT0, R24.2; no longer IC4RESET.BOOT0, R9.2
- net N$20: now also C5.1, C6.1, L3.1; no longer C1.1, C2.1, L1.1
- net N$21: now also IC2.1OUTR; no longer IC6.1OUTR
- net N$22: now also L3.2; no longer L1.2
- net N$23: now also R8.2; no longer R3.2
- net N$24: now also R16.1; no longer R14.1
- net N$25: now also R17.1, R18.2; no longer R5.1, R6.2
- net N$26: now also R19.1; no longer R15.1
- net N$27: now also IC2.1OUTG; no longer IC6.1OUTG
- net N$28: now also IC2.1OUTB; no longer IC6.1OUTB
- net N$29: now also IC2.2OUTR; no longer IC6.2OUTR
- net N$3: now also IC3PORTD/OSC.PD0/OSC<=, R25.2; no longer IC4PORTD/OSC.PD0/OSC<=, R10.2
- net N$30: now also IC2.2OUTG; no longer IC6.2OUTG
- net N$31: now also IC2.2OUTB; no longer IC6.2OUTB
- net N$32: now also R20.1; no longer R16.1
- net N$33: now also R21.1; no longer R17.1
- net N$34: now also R22.1; no longer R18.1
- net N$35: now also R23.1; no longer R19.1
- net N$36: now also IC2.VDD, R9.1; no longer IC6.VDD, R20.1
- net N$37: now also IC3PORTA_H.PA9, R6.2; no longer IC4PORTA_H.PA9, R22.2
- net N$38: now also IC3PORTA_H.PA10, R7.2; no longer IC4PORTA_H.PA10, R23.2
- net N$39: now also IC3PORTB_L.PB7, R14.1; no longer IC4PORTB_L.PB7, R25.1
- net N$4: now also IC3PORTD/OSC.PD1/OSC=>, R25.1; no longer IC4PORTD/OSC.PD1/OSC=>, R10.1
- net N$40: now also IC3PORTB_L.PB6, R13.1; no longer IC4PORTB_L.PB6, R24.1
- net N$41: now also R2.1; no longer R26.1
- net N$42: now also Q1.C; no longer Q2.C
- net N$5: now also IC3AN_POWER.VBAT; no longer IC4AN_POWER.VBAT
- net N$6: now also R10.2; no longer R1.2
- net N$7: now also S4.P; no longer S3.P
- net N$8: now also LED2.C, Q2.C; no longer LED1.C, Q1.C
- net SWDCLK: now also IC3PORTA_H.PA14; no longer IC4PORTA_H.PA14
- net SWDIO: now also IC3PORTA_H.PA13; no longer IC4PORTA_H.PA13
- net USART_RX: now also R7.1; no longer R23.1
- net USART_TX: now also R6.1; no longer R22.1
- net VOUT: now also IC4.VOUT; no longer IC5.VOUT
Other:
- moved on the sheet: C10, C19, C2, C20, C22, C23, C24, C3, C4, C5, C6, C7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

Commit message: wiring
Parts:
- added JP_LED_MCU, JP_LED_TM1809: (no value), SparkFun-Connectors:M03PTH
Connections:
- removed net LED_CTRL: IC2.DIN, R12.1
- removed net VOUT: C15.1, C16.1, IC4.VOUT
- new net LED_MCU: JP_LED_MCU.3
- new net LED_TM: IC2.DIN, JP_LED_TM1809.3, R12.1
- net 3.3V: now also C15.1, C16.1, C4.1, IC4.VOUT
- net 5V: now also JP_LED_MCU.1, JP_LED_TM1809.1; no longer C4.1
- net GND: now also JP_LED_MCU.2, JP_LED_TM1809.2
Other:
- moved on the sheet: C4

Commit message: nearly finish
Parts:
- added R28: 10K, SparkFun-Passives:RESISTOR0603-RES
Connections:
- new net N$44: C12.1, IC3RESET.NRST, R28.1
- net 3.3V: now also R28.2; no longer C12.1, IC3RESET.NRST
- net 5V: no longer C2.1, C3.1, R12.2
- net BTN_RELOAD: now also IC3PORTB_H.PB9
- net BTN_TRIGGER: now also IC3PORTB_L.PB5
- net BUZZER: now also IC3PORTA_L.PA2
- net DIP_SW1: now also IC3PORTB_H.PB14
- net DIP_SW2: now also IC3PORTB_H.PB13
- net DIP_SW3: now also IC3PORTB_H.PB12
- net GND: now also C2.1, C3.1, JP_LED_MCU.3, JP_LED_TM1809.3; no longer C2.2, C3.2, JP_LED_MCU.2, JP_LED_TM1809.2
- net IR_EMITTER: now also IC3PORTA_L.PA5
- net IR_RECEIVE1: now also IC3PORTB_H.PB10
- net IR_RECEIVE2: now also IC3PORTB_H.PB11
- net LED_MCU: now also IC3PORTB_H.PB8, JP_LED_MCU.2; no longer JP_LED_MCU.3
- net LED_TM: now also JP_LED_TM1809.2; no longer JP_LED_TM1809.3
- net N$36: now also C2.2, C3.2, R12.2
- net PWM_38K: now also IC3PORTA_L.PA6
Other:
- moved on the sheet: C2, C3

Commit message: finish wire
Parts:
- added Q3, Q4: 2N7002, SparkFun-DiscreteSemi:MOSFET-NCHANNELBSS138
- added R29, R30: 47K, SparkFun-Passives:RESISTOR0603-RES
- added R31, R32: 10K, SparkFun-Passives:RESISTOR0603-RES
- R13, R14: value 220R -> 100R
- R17: value 110K -> 110K(47K)
- R18: value 15K -> 15K(6.4K)
Connections:
- new net N$45: IC5.OUT, Q3.D, R30.1
- new net N$47: IC6.OUT, Q4.D, R29.1
- net 3.3V: now also Q3.G, Q4.G, R31.2, R32.2
- net 5V: now also R29.2, R30.2
- net IR_EMITTER: now also IC3PORTB_H.PB10; no longer IC3PORTA_L.PA5
- net IR_RECEIVE1: now also IC3PORTA_L.PA3, Q3.S, R31.1; no longer IC3PORTB_H.PB10, IC5.OUT
- net IR_RECEIVE2: now also Q4.S, R32.1; no longer IC6.OUT
Other:
- moved on the sheet: C23, C24, R26, R27

Commit message: finish
Parts:
- added R33, R34: 10K, SparkFun-Passives:RESISTOR0603-RES
- C22: device SparkFun-Passives:CAP0402-CAP -> SparkFun-Passives:CAP0603-CAP
- C24: device SparkFun-Passives:CAP0603-CAP -> SparkFun-Passives:CAP0402-CAP
- C3: value 1uf -> 100nf; device SparkFun-Passives:CAP0603-CAP -> SparkFun-Passives:CAP0402-CAP
- C4: value 100nf -> 10uf; device SparkFun-Passives:CAP0603-CAP -> SparkFun-Passives:CAP0402-CAP
- C5: value 100nf -> 1uf; device SparkFun-Passives:CAP0402-CAP -> SparkFun-Passives:CAP0603-CAP
- C6: value 10uf -> 100nf; device SparkFun-Passives:CAP0402-CAP -> SparkFun-Passives:CAP0603-CAP
- R25: value 1m -> 10K
- R26: value 100R -> 1m
- R28: value 10K -> 100R
- renumbered IR_LASER to JP4, JP1 to JP3, JP_LED_MCU to LED, JP_LED_TM1809 to JP2, L3 to L1, S4 to POWER, U$1 to J1
Connections:
- net BTN_TRIGGER renamed BTN_F1
- net 3.3V: now also C2.1, C24.1, R24.2; no longer C22.1, C4.1, R28.2
- net 5V: now also R28.2, R33.2, R34.2; no longer R26.2, R29.2, R30.2
- net GND: now also C2.2, C3.2, C5.1, C6.1, R25.1; no longer C2.1, C3.1, C5.2, C6.2, R24.1
- net I2C_SCL: now also R34.1
- net I2C_SDA: now also R33.1
- net IR_RECEIVE1: now also Q4.S, R32.1; no longer Q3.S, R31.1
- net IR_RECEIVE2: now also Q3.S, R31.1; no longer Q4.S, R32.1
- net N$11: now also C22.1, R27.1, R29.2; no longer C23.1, R26.1
- net N$12: now also C23.1, R28.1, R30.2; no longer C24.1, R27.1
- net N$2: now also R25.2; no longer R24.2
- net N$20: now also C3.1, C4.1; no longer C5.1, C6.1
- net N$3: now also R26.2; no longer R25.2
- net N$36: now also C5.2, C6.2; no longer C2.2, C3.2
- net N$4: now also R26.1; no longer R25.1
- net N$44: now also R24.1; no longer R28.1
- net N$45: now also Q4.D, R29.1; no longer Q3.D, R30.1
- net N$47: now also Q3.D, R30.1; no longer Q4.D, R29.1
Other:
- moved on the sheet: C2, C22, C23, C24, C3, C4, C5, C6, Q3, Q4, R24, R25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

Commit message: found some mistake, wait fixup
Parts:
- removed C3, C9: 100nf, SparkFun-Passives:CAP0402-CAP
- removed C4, C7, C8: 10uf, SparkFun-Passives:CAP0402-CAP
- added C25, C29: 100nf, SparkFun-Passives:CAP0603-CAP
- added C26, C27, C28: 10uf, SparkFun-Passives:CAP0603-CAP
Connections:
- net 5V: now also C27.2, C28.2, C29.2; no longer C7.1, C8.1, C9.1
- net GND: now also C25.2, C26.2, C27.1, C28.1, C29.1; no longer C3.2, C4.2, C7.2, C8.2, C9.2
- net N$20: now also C25.1, C26.1; no longer C3.1, C4.1
Changed lines of the file:
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@@
 <part name="R8" library="SparkFun-Passives" deviceset="RESISTOR" device="0603-RES" value="47k"/>
 <part name="GND10" library="SparkFun-Aesthetics" deviceset="GND" device=""/>
-<part name="C4" library="SparkFun-Passives" deviceset="CAP" device="0402-CAP" value="10uf"/>
 <part name="GND9" library="SparkFun-Aesthetics" deviceset="GND" device=""/>
 <part name="GND14" library="SparkFun-Aesthetics" deviceset="GND" device=""/>
 <part name="R17" library="SparkFun-Passives" deviceset="RESISTOR" device="0603-RES" value="110K(47K)"/>
 <part name="R18" library="SparkFun-Passives" deviceset="RESISTOR" device="0603-RES" value="15K(6.4K)"/>
-<part name="C8" library="SparkFun-Passives" deviceset="CAP" device="0402-CAP" value="10uf"/>
 <part name="GND15" library="SparkFun-Aesthetics" deviceset="GND" device=""/>
 <part name="SUPPLY11" library="SparkFun-Aesthetics" deviceset="5V" device=""/>
-<part name="C9" library="SparkFun-Passives" deviceset="CAP" device="0402-CAP" value="100nf"/>
 <part name="IC4" library="SparkFun-PowerIC" deviceset="XC6206" device=""/>
-<part name="C3" library="SparkFun-Passives" deviceset="CAP" device="0402-CAP" value="100nf"/>
-<part name="C7" library="SparkFun-Passives" deviceset="CAP" device="0402-CAP" value="10uf"/>
 <part name="GND20" library="SparkFun-Aesthetics" deviceset="GND" device=""/>
 <part name="SUPPLY12" library="SparkFun-Aesthetics" deviceset="5V" device=""/>
@@
 <part name="R33" library="SparkFun-Passives" deviceset="RESISTOR" device="0603-RES" value="10K"/>
 <part name="R34" library="SparkFun-Passives" deviceset="RESISTOR" device="0603-RES" value="10K"/>
+<part name="C25" library="SparkFun-Passives" deviceset="CAP" device="0603-CAP" value="100nf"/>
+<part name="C26" library="SparkFun-Passives" deviceset="CAP" device="0603-CAP" value="10uf"/>
+<part name="C27" library="SparkFun-Passives" deviceset="CAP" device="0603-CAP" value="10uf"/>
+<part name="C28" library="SparkFun-Passives" deviceset="CAP" device="0603-CAP" value="10uf"/>
+<part name="C29" library="SparkFun-Passives" deviceset="CAP" device="0603-CAP" value="100nf"/>
 </parts>
 <sheets>
@@
 <instance part="R8" gate="G$1" x="-99.06" y="213.36" rot="R90"/>
 <instance part="GND10" gate="1" x="-99.06" y="203.2"/>
-<instance part="C4" gate="G$1" x="-106.68" y="190.5"/>
 <instance part="GND9" gate="1" x="-106.68" y="180.34"/>
 <instance part="GND14" gate="1" x="-63.5" y="218.44"/>
 <instance part="R17" gate="G$1" x="-45.72" y="208.28" rot="R90"/>
 <instance part="R18" gate="G$1" x="-45.72" y="193.04" rot="R90"/>
-<instance part="C8" gate="G$1" x="-25.4" y="200.66"/>
 <instance part="GND15" gate="1" x="-45.72" y="182.88"/>
 <instance part="SUPPLY11" gate="G$1" x="-15.24" y="215.9"/>
-<instance part="C9" gate="G$1" x="-15.24" y="200.66"/>
 <instance part="IC4" gate="G$1" x="43.18" y="203.2" rot="MR90"/>
-<instance part="C3" gate="G$1" x="-114.3" y="190.5"/>
-<instance part="C7" gate="G$1" x="-35.56" y="200.66"/>
 <instance part="GND20" gate="1" x="43.18" y="182.88"/>
 <instance part="SUPPLY12" gate="G$1" x="10.16" y="205.74"/>
@@
 <instance part="R33" gate="G$1" x="-149.86" y="127" rot="R90"/>
 <instance part="R34" gate="G$1" x="-142.24" y="127" rot="R90"/>
+<instance part="C25" gate="G$1" x="-114.3" y="190.5"/>
+<instance part="C26" gate="G$1" x="-106.68" y="190.5"/>
+<instance part="C27" gate="G$1" x="-35.56" y="203.2" rot="R180"/>
+<instance part="C28" gate="G$1" x="-25.4" y="203.2" rot="R180"/>
+<instance part="C29" gate="G$1" x="-15.24" y="203.2" rot="R180"/>
 </instances>
 <busses>
@@
 </segment>
 <segment>
-<wire x1="-114.3" y1="187.96" x2="-114.3" y2="185.42" width="0.1524" layer="91"/>
-<wire x1="-114.3" y1="185.42" x2="-106.68" y2="185.42" width="0.1524" layer="91"/>
-<pinref part="C4" gate="G$1" pin="2"/>
-<wire x1="-106.68" y1="185.42" x2="-106.68" y2="187.96" width="0.1524" layer="91"/>
 <pinref part="JP3" gate="G$1" pin="1"/>
 <wire x1="-142.24" y1="195.58" x2="-142.24" y2="185.42" width="0.1524" layer="91"/>
 <wire x1="-142.24" y1="185.42" x2="-114.3" y2="185.42" width="0.1524" layer="91"/>
+<pinref part="GND9" gate="1" pin="GND"/>
+<wire x1="-114.3" y1="185.42" x2="-106.68" y2="185.42" width="0.1524" layer="91"/>
+<wire x1="-106.68" y1="182.88" x2="-106.68" y2="185.42" width="0.1524" layer="91"/>
+<pinref part="C25" gate="G$1" pin="2"/>
+<wire x1="-114.3" y1="185.42" x2="-114.3" y2="187.96" width="0.1524" layer="91"/>
 <junction x="-114.3" y="185.42"/>
-<pinref part="GND9" gate="1" pin="GND"/>
-<wire x1="-106.68" y1="182.88" x2="-106.68" y2="185.42" width="0.1524" layer="91"/>
+<pinref part="C26" gate="G$1" pin="2"/>
+<wire x1="-106.68" y1="187.96" x2="-106.68" y2="185.42" width="0.1524" layer="91"/>
 <junction x="-106.68" y="185.42"/>
-<pinref part="C3" gate="G$1" pin="2"/>
 </segment>
 <segment>
@@
 <segment>
 <pinref part="R18" gate="G$1" pin="1"/>
-<wire x1="-45.72" y1="187.96" x2="-35.56" y2="187.96" width="0.1524" layer="91"/>
-<wire x1="-35.56" y1="187.96" x2="-35.56" y2="198.12" width="0.1524" layer="91"/>
-<pinref part="C8" gate="G$1" pin="2"/>
-<wire x1="-35.56" y1="187.96" x2="-25.4" y2="187.96" width="0.1524" layer="91"/>
-<wire x1="-25.4" y1="187.96" x2="-25.4" y2="198.12" width="0.1524" layer="91"/>
-<junction x="-35.56" y="187.96"/>
 <pinref part="GND15" gate="1" pin="GND"/>
 <wire x1="-45.72" y1="185.42" x2="-45.72" y2="187.96" width="0.1524" layer="91"/>
 <junction x="-45.72" y="187.96"/>
-<pinref part="C9" gate="G$1" pin="2"/>
+<wire x1="-15.24" y1="187.96" x2="-25.4" y2="187.96" width="0.1524" layer="91"/>
+<pinref part="C27" gate="G$1" pin="1"/>
+<wire x1="-25.4" y1="187.96" x2="-35.56" y2="187.96" width="0.1524" layer="91"/>
+<wire x1="-35.56" y1="187.96" x2="-45.72" y2="187.96" width="0.1524" layer="91"/>
+<wire x1="-35.56" y1="198.12" x2="-35.56" y2="187.96" width="0.1524" layer="91"/>
+<junction x="-35.56" y="187.96"/>
+<pinref part="C28" gate="G$1" pin="1"/>
+<wire x1="-25.4" y1="198.12" x2="-25.4" y2="187.96" width="0.1524" layer="91"/>
+<junction x="-25.4" y="187.96"/>
+<pinref part="C29" gate="G$1" pin="1"/>
 <wire x1="-15.24" y1="198.12" x2="-15.24" y2="187.96" width="0.1524" layer="91"/>
-<wire x1="-15.24" y1="187.96" x2="-25.4" y2="187.96" width="0.1524" layer="91"/>
-<junction x="-25.4" y="187.96"/>
-<pinref part="C7" gate="G$1" pin="2"/>
 </segment>
 <segment>
@@
 <pinref part="R17" gate="G$1" pin="2"/>
 <wire x1="-45.72" y1="213.36" x2="-35.56" y2="213.36" width="0.1524" layer="91"/>
+<junction x="-45.72" y="213.36"/>
+<pinref part="SUPPLY11" gate="G$1" pin="5V"/>
 <wire x1="-35.56" y1="213.36" x2="-25.4" y2="213.36" width="0.1524" layer="91"/>
 <wire x1="-25.4" y1="213.36" x2="-15.24" y2="213.36" width="0.1524" layer="91"/>
-<junction x="-45.72" y="213.36"/>
+<wire x1="-15.24" y1="213.36" x2="-15.24" y2="215.9" width="0.1524" layer="91"/>
+<pinref part="D1" gate="G$1" pin="C"/>
+<pinref part="C27" gate="G$1" pin="2"/>
 <wire x1="-35.56" y1="205.74" x2="-35.56" y2="213.36" width="0.1524" layer="91"/>
 <junction x="-35.56" y="213.36"/>
-<pinref part="C8" gate="G$1" pin="1"/>
+<pinref part="C28" gate="G$1" pin="2"/>
 <wire x1="-25.4" y1="205.74" x2="-25.4" y2="213.36" width="0.1524" layer="91"/>
 <junction x="-25.4" y="213.36"/>
-<pinref part="SUPPLY11" gate="G$1" pin="5V"/>
-<wire x1="-15.24" y1="213.36" x2="-15.24" y2="215.9" width="0.1524" layer="91"/>
-<pinref part="C9" gate="G$1" pin="1"/>
+<pinref part="C29" gate="G$1" pin="2"/>
 <wire x1="-15.24" y1="205.74" x2="-15.24" y2="213.36" width="0.1524" layer="91"/>
 <junction x="-15.24" y="213.36"/>
-<pinref part="C7" gate="G$1" pin="1"/>
-<pinref part="D1" gate="G$1" pin="C"/>
 </segment>
 <segment>
@@
 <pinref part="F1" gate="G$1" pin="2"/>
 <wire x1="-116.84" y1="198.12" x2="-114.3" y2="198.12" width="0.1524" layer="91"/>
-<pinref part="C4" gate="G$1" pin="1"/>
 <wire x1="-114.3" y1="198.12" x2="-106.68" y2="198.12" width="0.1524" layer="91"/>
-<wire x1="-106.68" y1="195.58" x2="-106.68" y2="198.12" width="0.1524" layer="91"/>
-<wire x1="-114.3" y1="195.58" x2="-114.3" y2="198.12" width="0.1524" layer="91"/>
-<junction x="-114.3" y="198.12"/>
 <wire x1="-106.68" y1="198.12" x2="-106.68" y2="220.98" width="0.1524" layer="91"/>
 <junction x="-106.68" y="198.12"/>
@@
 <junction x="-106.68" y="220.98"/>
 <wire x1="-106.68" y1="198.12" x2="-88.9" y2="198.12" width="0.1524" layer="91"/>
-<pinref part="C3" gate="G$1" pin="1"/>
 <pinref part="L1" gate="G$1" pin="1"/>
-</segment>
-</net>
+<pinref part="C25" gate="G$1" pin="1"/>
+<wire x1="-114.3" y1="195.58" x2="-114.3" y2="198.12" width="0.1524" layer="91"/>
+<junction x="-114.3" y="198.12"/>
+<pinref part="C26" gate="G$1" pin="1"/>
+<wire x1="-106.68" y1="195.58" x2="-106.68" y2="198.12" width="0.1524" layer="91"/>
+</segment>
+</net>

Commit message: modify some packages
Parts:
- removed C16, C17, C18, C21: 100nf, SparkFun-Passives:CAP0402-CAP
- removed C24: 4.7uf, SparkFun-Passives:CAP0402-CAP
- removed U1: 74LVC1G08SE-7, SparkFun-DigitalIC:7408SE
- added C3, C7: 1uf, SparkFun-Passives:CAP0603-CAP
- added C4, C8, C9: 100nf, SparkFun-Passives:CAP0603-CAP
- added U$1: SN74LVC1G08, SparkFun-DigitalIC:SN74LVC1G08
- C10: value 1uf -> 100nf; device SparkFun-Passives:CAP0402-CAP -> SparkFun-Passives:CAP0603-CAP
- C11: device SparkFun-Passives:CAP0402-CAP -> SparkFun-Passives:CAP0603-CAP
- C15: value 1uf -> 4.7uf; device SparkFun-Passives:CAP0402-CAP -> SparkFun-Passives:CAP0603-CAP
Connections:
- net 3.3V: now also C10.1, C11.1, C7.1, C8.1, C9.1, U$1.+V; no longer C16.1, C17.1, C18.1, C21.1, C24.1, U1.VCC
- net 5V: now also C3.1, C4.1; no longer C10.1, C11.1
- net GND: now also C3.2, C4.2, C7.2, C8.2, C9.2, U$1.GND; no longer C16.2, C17.2, C18.2, C21.2, C24.2, U1.GND
- net I2C_SCL: now also IC3PORTB_L.PB6; no longer J1.2
- net I2C_SDA: now also IC3PORTB_L.PB7; no longer J1.3
- net IR_EMITTER: now also U$1.A; no longer U1.A
- net N$39: now also J1.3; no longer IC3PORTB_L.PB7
- net N$40: now also J1.2; no longer IC3PORTB_L.PB6
- net N$6: now also U$1.Y; no longer U1.Y
- net PWM_38K: now also U$1.B; no longer U1.B
Other:
- moved on the sheet: C10, C11, C15, R13, R14
