File: hardware/v0.1/1.sch (EAGLE design)
At the start: 95 parts, among them IC1 FP6291, IC2 TM1809, IC3 STM32F10XCXT6, IC5 TSOP34830, IC6 TSOP34830, J1 RJ9PTH, Q1 8050, Q2 8050, Q3 2N7002, Q4 2N7002, Y1 8M

Commit message: update silkscreen
Parts:
- removed C25, C29: 100nf, SparkFun-Passives:CAP0603-CAP
- removed C26, C27, C28: 10uf, SparkFun-Passives:CAP0603-CAP
- removed U$1: SN74LVC1G08, SparkFun-DigitalIC:SN74LVC1G08
- added C16, C17, C18, C21: 100nf, SparkFun-Passives:CAP0603-CAP
- added C24: 4.7uf, SparkFun-Passives:CAP0603-CAP
- added IC7: TSOP34830, vishay-1:TSOP34830
- C10: value 100nf -> 1uf
- C15: value 4.7uf -> 1uf
- C3: value 1uf -> 100nf
- C4, C8: value 100nf -> 10uf
- C7: value 1uf -> 10uf
- IC1: value FP6291 -> SN74LVC1G08; device eagle_lib_lishen:FP6291 -> SparkFun-DigitalIC:SN74LVC1G08
- IC2: value TM1809 -> FP6291; device eagle_lib_lishen:TM1809 -> eagle_lib_lishen:FP6291
- IC3: value STM32F10XCXT6 -> TM1809; device stm32:STM32F10XCXT6 -> eagle_lib_lishen:TM1809
- IC4: value (none) -> STM32F10XCXT6; device SparkFun-PowerIC:XC6206 -> stm32:STM32F10XCXT6
- IC5: value TSOP34830 -> (none); device vishay-1:TSOP34830 -> SparkFun-PowerIC:XC6206
- R10: value 2.2K -> 220R
- R11: value 51 -> 220R; device SparkFun-Resistors:RESISTOR1206 -> SparkFun-Passives:RESISTOR0603-RES
- R12: value 10K -> 47k
- R14: value 100R -> 2.2K
- R15: value 10K -> 51; device SparkFun-Passives:RESISTOR0603-RES -> SparkFun-Resistors:RESISTOR1206
- R16, R5: value 470R -> 10K
- R17: value 110K(47K) -> 10K
- R18: value 15K(6.4K) -> 470R
- R19: value 470R -> 110K(47K)
- R20: value 470R -> 15K(6.4K)
- R24, R25: value 10K -> 470R
- R26: value 1m -> 10K
- R27: value 100R -> 10K
- R28: value 100R -> 1m
- R29, R30: value 47K -> 100R
- R3, R4: value 470R -> 100R
- R31, R32: value 10K -> 47K
- R6: value 220R -> 10K
- R7: value 220R -> 470R
- R8: value 47k -> 470R
- R9: value 100R -> 470R
- renumbered LED to JP1, POWER to S4, SWD to JP7, UPDATE to JP5, USART to JP6
Connections:
- net 3.3V: now also C16.1, C17.1, C18.1, C21.1, C24.1, IC1.+V, IC4AN_POWER.VDDA, IC4POWER.VDD_1, IC4POWER.VDD_2, IC4POWER.VDD_3, IC5.VOUT, R26.2, R33.2, R34.2; no longer C10.1, C11.1, C7.1, C8.1, C9.1, IC3AN_POWER.VDDA, IC3POWER.VDD_1, IC3POWER.VDD_2, IC3POWER.VDD_3, IC4.VOUT, R24.2, R31.2, R32.2, U$1.+V
- net 5V: now also C10.1, C11.1, C7.2, C8.2, C9.2, IC5.VIN, R13.2, R15.2, R18.2, R24.2, R25.2, R29.2, R30.2, R6.2, R7.2, R8.2; no longer C27.2, C28.2, C29.2, C3.1, C4.1, IC4.VIN, R11.2, R16.2, R17.2, R20.2, R27.2, R28.2, R3.2, R33.2, R34.2, R4.2
- net BTN_F1: now also IC4PORTB_L.PB5; no longer IC3PORTB_L.PB5
- net BTN_RELOAD: now also IC4PORTB_H.PB9; no longer IC3PORTB_H.PB9
- net BUZZER: now also IC4PORTA_L.PA2; no longer IC3PORTA_L.PA2
- net DIP_SW1: now also IC4PORTB_H.PB14; no longer IC3PORTB_H.PB14
- net DIP_SW2: now also IC4PORTB_H.PB13; no longer IC3PORTB_H.PB13
- net DIP_SW3: now also IC4PORTB_H.PB12; no longer IC3PORTB_H.PB12
- net GND: now also C16.2, C17.2, C18.2, C21.2, C24.2, C7.1, C8.1, C9.1, IC3.GND, IC4AN_POWER.VSSA, IC4POWER.VSS_1, IC4POWER.VSS_2, IC4POWER.VSS_3, IC5.VSS, IC7.GND, R12.1, R17.2, R20.1, R27.1; no longer C25.2, C26.2, C27.1, C28.1, C29.1, C7.2, C8.2, C9.2, IC3AN_POWER.VSSA, IC3POWER.VSS_1, IC3POWER.VSS_2, IC3POWER.VSS_3, IC4.VSS, IC5.GND, R15.2, R18.1, R25.1, R8.1, U$1.GND
- net I2C_SCL: now also IC4PORTB_L.PB6, R4.2, R6.1; no longer IC3PORTB_L.PB6, R13.2, R34.1
- net I2C_SDA: now also IC4PORTB_L.PB7, R3.2, R5.1; no longer IC3PORTB_L.PB7, R14.2, R33.1
- net IR_EMITTER: now also IC1.A, IC4PORTB_H.PB10; no longer IC3PORTB_H.PB10, U$1.A
- net IR_RECEIVE1: now also IC4PORTA_L.PA3, R34.1; no longer IC3PORTA_L.PA3, R32.1
- net IR_RECEIVE2: now also IC4PORTB_H.PB11, R33.1; no longer IC3PORTB_H.PB11, R31.1
- net LED_MCU: now also IC4PORTB_H.PB8; no longer IC3PORTB_H.PB8
- net LED_TM: now also IC3.DIN, R16.1; no longer IC2.DIN, R12.1
- net N$1: now also IC4PORTB_L.PB2, R17.1; no longer IC3PORTB_L.PB2, R15.1
- net N$11: now also IC6.VS, R29.1, R31.2; no longer IC5.VS, R27.1, R29.2
- net N$12: now also IC7.VS, R30.1, R32.2; no longer IC6.VS, R28.1, R30.2
- net N$13: now also IC3.3OUTR; no longer IC2.3OUTR
- net N$14: now also R15.1; no longer R11.1
- net N$15: now also IC3.3OUTG; no longer IC2.3OUTG
- net N$16: now also IC3.3OUTB; no longer IC2.3OUTB
- net N$17: now also R9.1; no longer R5.1
- net N$18: now also R8.1; no longer R4.1
- net N$19: now also R7.1; no longer R3.1
- net N$2: now also IC4RESET.BOOT0, R27.2; no longer IC3RESET.BOOT0, R25.2
- net N$20: now also C3.1, C4.1, IC2.EN, IC2.VCC; no longer C25.1, C26.1, IC1.EN, IC1.VCC
- net N$21: now also IC3.1OUTR; no longer IC2.1OUTR
- net N$22: now also IC2.LX; no longer IC1.LX
- net N$23: now also IC2.OC, R12.2; no longer IC1.OC, R8.2
- net N$24: now also R18.1; no longer R16.1
- net N$25: now also IC2.FB, R19.1, R20.2; no longer IC1.FB, R17.1, R18.2
- net N$26: now also R21.1; no longer R19.1
- net N$27: now also IC3.1OUTG; no longer IC2.1OUTG
- net N$28: now also IC3.1OUTB; no longer IC2.1OUTB
- net N$29: now also IC3.2OUTR; no longer IC2.2OUTR
- net N$3: now also IC4PORTD/OSC.PD0/OSC<=, R28.2; no longer IC3PORTD/OSC.PD0/OSC<=, R26.2
- net N$30: now also IC3.2OUTG; no longer IC2.2OUTG
- net N$31: now also IC3.2OUTB; no longer IC2.2OUTB
- net N$32: now also R22.1; no longer R20.1
- net N$33: now also R23.1; no longer R21.1
- net N$34: now also R24.1; no longer R22.1
- net N$35: now also R25.1; no longer R23.1
- net N$36: now also IC3.VDD, R13.1, R16.2; no longer IC2.VDD, R12.2, R9.1
- net N$37: now also IC4PORTA_H.PA9, R10.2; no longer IC3PORTA_H.PA9, R6.2
- net N$38: now also IC4PORTA_H.PA10, R11.2; no longer IC3PORTA_H.PA10, R7.2
- net N$39: now also R3.1; no longer R14.1
- net N$4: now also IC4PORTD/OSC.PD1/OSC=>, R28.1; no longer IC3PORTD/OSC.PD1/OSC=>, R26.1
- net N$40: now also R4.1; no longer R13.1
- net N$44: now also IC4RESET.NRST, R26.1; no longer IC3RESET.NRST, R24.1
- net N$45: now also IC6.OUT, R31.1; no longer IC5.OUT, R29.1
- net N$47: now also IC7.OUT, R32.1; no longer IC6.OUT, R30.1
- net N$5: now also IC4AN_POWER.VBAT; no longer IC3AN_POWER.VBAT
- net N$6: now also IC1.Y, R14.2; no longer R10.2, U$1.Y
- net N$9: now also R14.1; no longer R10.1
- net PWM_38K: now also IC1.B, IC4PORTA_L.PA6; no longer IC3PORTA_L.PA6, U$1.B
- net SWDCLK: now also IC4PORTA_H.PA14; no longer IC3PORTA_H.PA14
- net SWDIO: now also IC4PORTA_H.PA13; no longer IC3PORTA_H.PA13
- net USART_RX: now also R11.1; no longer R7.1
- net USART_TX: now also R10.1; no longer R6.1
Other:
- moved on the sheet: C10, C11, C15, C3, C4, C7, C8, C9, IC6, R10, R11, R12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
