File: hardware/v0.2/2_main.brd (EAGLE design)
At the start: 72 x 45 mm, 72 parts, among them IC1 SN74LVC1G08, IC2 FP6291, IC4 STM32F10XCXT6, J1 RJ9PTH, Q2 8050, Q3 MOSFET-NCHANNELBSS138, Q4 MOSFET-NCHANNELBSS138, Y1 8M

Commit message: update sch
Parts:
- removed IC4: STM32F10XCXT6, stm32:TQFP48
- added JP8: (no value), SparkFun-Connectors:1X08
- added U1: STM32F10XRXT6, stm32:TQFP64
- moved J1 1.00 mm to (61.3, 18.1)
Connections:
- removed net LED_MCU: IC4.45
- removed net N$37: IC4.30, R10.2
- removed net N$38: IC4.31, R11.2
- new net LCD_CLK: JP8.7
- new net LCD_CS: JP8.5
- new net LCD_DC: JP8.6
- new net LCD_MOSI: JP8.8
- new net LCD_PWR: JP8.4
- new net LCD_VBAT: JP8.1
- new net N$27: R10.2, U1.42
- new net N$28: R11.2, U1.43
- new net VDD: JP8.3
- net 3.3V: now also U1.13, U1.19, U1.32, U1.48, U1.64; no longer IC4.24, IC4.36, IC4.48, IC4.9
- net BTN_FIRE: no longer IC4.41
- net BTN_RELOAD: no longer IC4.46
- net GND: now also JP8.2, U1.12, U1.18, U1.31, U1.47, U1.63; no longer IC4.23, IC4.35, IC4.47, IC4.8
- net IR_EMITTER: no longer IC4.12
- net N$1: now also U1.28; no longer IC4.20
- net N$2: now also U1.60; no longer IC4.44
- net N$3: now also U1.5; no longer IC4.5
- net N$4: now also U1.6; no longer IC4.6
- net N$44: now also U1.7; no longer IC4.7
- net N$5: now also U1.1; no longer IC4.1
- net PORT_RX: no longer IC4.22
- net PORT_TX: no longer IC4.21
- net PWM_38K: no longer IC4.16
- net SWDCLK: now also U1.49; no longer IC4.37
- net SWDIO: now also U1.46; no longer IC4.34
Routing:
- net 3.3V: track 102.5 -> 85.2 mm
- net N$2: track 27.7 -> 20.0 mm
- net BTN_FIRE: track 44.4 -> 37.2 mm
- net GND: track 418.5 -> 412.1 mm
- net N$1: track 6.25 -> 0.00 mm
- net SWDCLK: track 14.8 -> 8.60 mm
- net N$37: track 6.08 -> 0.00 mm
- net N$38: track 5.25 -> 0.00 mm
- net SWDIO: track 13.8 -> 9.34 mm
- net PWM_38K: track 8.32 -> 4.57 mm
- net N$4: track 11.9 -> 8.47 mm
- net N$3: track 11.9 -> 8.47 mm
- net BTN_RELOAD: track 56.5 -> 53.8 mm
- net N$44: track 9.32 -> 7.17 mm
- net N$5: track 2.96 -> 1.40 mm
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
Commit message: update sch
Parts:
- removed JP3: M02PTH, SparkFun-Connectors:1X02
- removed JP4: (no value), SparkFun-Connectors:1X03
- added C22: 100nf, SparkFun-Passives:0603-CAP
- added JP1: M02POLAR, SparkFun-Connectors:MOLEX-1X2
- added Q5: 8550, SparkFun-DiscreteSemi:SOT23
- added R16: 51, SparkFun-Passives:0603-RES
- added R18: 1K, SparkFun-Passives:0603-RES
- added R21, R22: 0R, SparkFun-Passives:0603-RES
- added R23: 10K, SparkFun-Passives:0603-RES
- R15: value 51 -> 1K; device SparkFun-Resistors:1206 -> SparkFun-Passives:0603-RES
- moved R15 127.0 mm to (-43.0, -89.0), turned to 0 degrees
- moved U1 78.5 mm to (23.0, 17.0), turned to 180 degrees
Connections:
- removed net FLASH_SCK: U$1.6
- removed net LCD_CS: JP8.5
- removed net LCD_VBAT: JP8.1
- new net FLASH_CLK: U$1.6, U1.34
- new net IR_EMMITER: U1.29
- new net N$29: Q5.1, R15.2, R23.1
- new net N$30: C22.1, R18.2, R21.1
- new net N$31: R22.2, U1.20
- new net N$32: JP8.1, Q5.3
- new net V_BATT: C3.1, C4.1, F1.2, IC2.4, IC2.5, L1.P$1, Q5.2, R23.2
- net 5V: now also R16.2; no longer R15.2
- net AUDIO_OUT: now also R21.2, R22.1
- net FLASH_CS: now also U1.33
- net FLASH_MISO: now also U1.35
- net FLASH_MOSI: now also U1.36
- net GND: now also C22.2, JP1.1; no longer JP3.1, JP4.3
- net LCD_CLK: now also U1.21
- net LCD_DC: now also U1.22
- net LCD_MOSI: now also U1.23
- net LCD_PWR: now also R15.1, U1.30; no longer JP8.4
- net N$14: now also R18.1; no longer JP4.1, LED2.A, R15.1
- net N$20: now also LED2.A, R16.1; no longer C3.1, C4.1, F1.2, IC2.4, IC2.5, L1.P$1
- net N$7: now also JP1.2; no longer JP3.2
- net N$8: no longer JP4.2
- net PORT_RX: now also U1.52
- net PORT_TX: now also U1.51
- net PWM_38K: now also U1.27
Routing:
- net N$20: track 29.8 -> 0.00 mm
- net N$14: track 14.4 -> 0.00 mm
- net GND: track 412.1 -> 407.0 mm
- net N$8: track 17.3 -> 15.8 mm
Other:
- board text removed: "FIRE"
- board text removed: "Function"

Commit message: add mirco sd socket
Parts:
- removed JP8: (no value), SparkFun-Connectors:1X08
- removed Q5: 8550, SparkFun-DiscreteSemi:SOT23
- removed R15: 1K, SparkFun-Passives:0603-RES
- added D3: 1N5819, SparkFun-DiscreteSemi:SOD-323
- added JP3: (no value), SparkFun-Connectors:MOLEX-1X6
- added Q1: PMOS, SparkFun-DiscreteSemi:SOT23-3
- added SD1: MICROSD_YOUXIN, eagle_lib_lishen:MICRO_SD_YOUXIN
Connections:
- new net SD_CLK: SD1.5, U1.55
- new net SD_CS: SD1.2, U1.58
- new net SD_MISO: SD1.7, U1.56
- new net SD_MOSI: SD1.3, U1.57
- net 3.3V: now also SD1.4
- net GND: now also JP3.2, SD1.6; no longer JP8.2
- net LCD_CLK: now also JP3.5; no longer JP8.7
- net LCD_DC: now also JP3.4; no longer JP8.6
- net LCD_MOSI: now also JP3.6; no longer JP8.8
- net LCD_PWR: now also Q1.1, R23.1; no longer R15.1
- net N$29: now also D3.1, JP3.1; no longer Q5.1, R15.2, R23.1
- net N$32: now also D3.2, Q1.3; no longer JP8.1, Q5.3
- net VDD: now also JP3.3; no longer JP8.3
- net V_BATT: now also Q1.2; no longer Q5.2
Changed lines of the file:
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@@
 <element name="S6" library="SparkFun-Electromechanical" package="TACTILE-SWITCH-1101NE" value="SWITCH-MOMENTARY-2-SMD-1101NE" x="36" y="8"/>
 <element name="U1" library="stm32" package="TQFP64" value="STM32F10XRXT6" x="23" y="17" rot="R180"/>
-<element name="JP8" library="SparkFun-Connectors" package="1X08" value="" x="-35" y="-68"/>
 <element name="JP1" library="SparkFun-Connectors" package="MOLEX-1X2" value="M02POLAR" x="68" y="40" rot="R90"/>
 <element name="R18" library="SparkFun-Passives" package="0603-RES" value="1K" x="-35" y="-74"/>
@@
 <element name="R22" library="SparkFun-Passives" package="0603-RES" value="0R" x="-35" y="-83"/>
 <element name="R16" library="SparkFun-Passives" package="0603-RES" value="51" x="-35" y="-86"/>
-<element name="R15" library="SparkFun-Passives" package="0603-RES" value="1K" x="-43" y="-89"/>
-<element name="Q5" library="SparkFun-DiscreteSemi" package="SOT23" value="8550" x="-47" y="-88">
-<attribute name="PROD_ID" value="TRANS-09245" x="-47" y="-88" size="1.778" layer="27" display="off"/>
+<element name="R23" library="SparkFun-Passives" package="0603-RES" value="10K" x="-47" y="-92"/>
+<element name="Q1" library="SparkFun-DiscreteSemi" package="SOT23-3" value="PMOS" x="-51" y="-92"/>
+<element name="D3" library="SparkFun-DiscreteSemi" package="SOD-323" value="1N5819" x="-55" y="-91">
+<attribute name="PROD_ID" value="DIO-11623" x="-55" y="-91" size="1.778" layer="27" display="off"/>
 </element>
-<element name="R23" library="SparkFun-Passives" package="0603-RES" value="10K" x="-47" y="-92"/>
+<element name="JP3" library="SparkFun-Connectors" package="MOLEX-1X6" value="" x="-55" y="-97"/>
+<element name="SD1" library="eagle_lib_lishen" package="MICRO_SD_YOUXIN" value="MICROSD_YOUXIN" x="-66" y="-94"/>
 </elements>
 <signals>
@@
 <contactref element="U1" pad="19"/>
 <contactref element="U1" pad="32"/>
+<contactref element="SD1" pad="4"/>
+<wire x1="-23.25" y1="-44.8" x2="-67.05" y2="-79.5" width="0" layer="19" extent="1-1"/>
 <wire x1="-21.55" y1="-41.8" x2="-23.25" y2="-44.8" width="0" layer="19" extent="1-1"/>
 <wire x1="-23.405" y1="-33.9838" x2="-21.55" y2="-41.8" width="0" layer="19" extent="1-1"/>
@@
 </signal>
 <signal name="GND">
-<contactref element="R17" pad="2"/>
 <contactref element="C12" pad="2"/>
 <contactref element="R27" pad="1"/>
@@
 <wire x1="12.75" y1="12.75" x2="11" y2="14.5" width="0.254" layer="1"/>
 <wire x1="11" y1="14.5" x2="11" y2="15.85" width="0.254" layer="1"/>
-<wire x1="11" y1="15.85" x2="11.15" y2="16" width="0.254" layer="1"/>
 <wire x1="18.25" y1="14.75" x2="17" y2="13.5" width="0.254" layer="1"/>
 <via x="17" y="13.5" extent="1-16" drill="0.5"/>
@@
 <wire x1="14" y1="21" x2="11" y2="18" width="0.254" layer="1"/>
 <wire x1="11" y1="18" x2="11" y2="16.15" width="0.254" layer="1"/>
-<wire x1="11" y1="16.15" x2="11.15" y2="16" width="0.254" layer="1"/>
 <contactref element="C17" pad="2"/>
 <contactref element="C18" pad="2"/>
@@
 <contactref element="U1" pad="63"/>
 <contactref element="U1" pad="18"/>
-<contactref element="JP8" pad="2"/>
 <contactref element="JP1" pad="1"/>
 <contactref element="C22" pad="2"/>
-<wire x1="-32.46" y1="-68" x2="-34.15" y2="-80" width="0" layer="19" extent="1-1"/>
-<wire x1="-21.55" y1="-44.8" x2="-32.46" y2="-68" width="0" layer="19" extent="1-1"/>
+<contactref element="JP3" pad="2"/>
+<contactref element="SD1" pad="6"/>
+<contactref element="R17" pad="2"/>
+<wire x1="-69.25" y1="-79.5" x2="-52.46" y2="-97" width="0" layer="19" extent="1-1"/>
+<wire x1="-34.15" y1="-80" x2="-52.46" y2="-97" width="0" layer="19" extent="1-1"/>
+<wire x1="-21.55" y1="-44.8" x2="-34.15" y2="-80" width="0" layer="19" extent="1-1"/>
 <wire x1="-19.595" y1="-39.2162" x2="-21.55" y2="-44.8" width="0" layer="19" extent="1-1"/>
 <wire x1="-17.55" y1="-28.6" x2="-19.595" y2="-39.2162" width="0" layer="19" extent="1-1"/>
@@
 <wire x1="19.75" y1="22.7" x2="20.5" y2="24.5" width="0" layer="19" extent="1-1"/>
 <wire x1="20.85" y1="21.35" x2="19.75" y2="22.7" width="0" layer="19" extent="1-16"/>
+<wire x1="11.15" y1="16" x2="11" y2="15.85" width="0" layer="19" extent="1-1"/>
+<wire x1="11" y1="16.15" x2="11.15" y2="16" width="0" layer="19" extent="1-1"/>
 <wire x1="17.3" y1="13.75" x2="17" y2="13.5" width="0" layer="19" extent="1-1"/>
 <wire x1="28.7" y1="18.75" x2="29.25" y2="19.25" width="0" layer="19" extent="1-1"/>
@@
 <wire x1="23.5" y1="7.35" x2="17.3" y2="15.75" width="0" layer="19" extent="1-1"/>
 </signal>
-<signal name="VDD">
-<contactref element="JP8" pad="3"/>
-</signal>
 <signal name="LCD_DC">
-<contactref element="JP8" pad="6"/>
 <contactref element="U1" pad="22"/>
-<wire x1="24.25" y1="22.7" x2="-22.3" y2="-68" width="0" layer="19" extent="1-1"/>
+<contactref element="JP3" pad="4"/>
+<wire x1="24.25" y1="22.7" x2="-47.38" y2="-97" width="0" layer="19" extent="1-1"/>
 </signal>
 <signal name="LCD_CLK">
-<contactref element="JP8" pad="7"/>
 <contactref element="U1" pad="21"/>
-<wire x1="24.75" y1="22.7" x2="-19.76" y2="-68" width="0" layer="19" extent="1-1"/>
+<contactref element="JP3" pad="5"/>
+<wire x1="24.75" y1="22.7" x2="-44.84" y2="-97" width="0" layer="19" extent="1-1"/>
 </signal>
 <signal name="LCD_MOSI">
-<contactref element="JP8" pad="8"/>
 <contactref element="U1" pad="23"/>
-<wire x1="23.75" y1="22.7" x2="-17.22" y2="-68" width="0" layer="19" extent="1-1"/>
+<contactref element="JP3" pad="6"/>
+<wire x1="23.75" y1="22.7" x2="-42.3" y2="-97" width="0" layer="19" extent="1-1"/>
 </signal>
 <signal name="V_BATT">
@@
 <contactref element="C4" pad="1"/>
 <contactref element="L1" pad="P$1"/>
-<contactref element="Q5" pad="2"/>
 <contactref element="R23" pad="2"/>
-<wire x1="-46.05" y1="-89.1" x2="-46.15" y2="-92" width="0" layer="19" extent="1-1"/>
-<wire x1="56.85" y1="28" x2="-46.05" y2="-89.1" width="0" layer="19" extent="1-1"/>
+<contactref element="Q1" pad="2"/>
+<wire x1="-46.15" y1="-92" x2="-50.05" y2="-93" width="0" layer="19" extent="1-1"/>
+<wire x1="56.85" y1="28" x2="-46.15" y2="-92" width="0" layer="19" extent="1-1"/>
 <wire x1="56.85" y1="30.5" x2="56.85" y2="28" width="0" layer="19" extent="1-1"/>
 <wire x1="55.8001" y1="33.05" x2="56.85" y2="30.5" width="0" layer="19" extent="1-1"/>
@@
 </signal>
 <signal name="LCD_PWR">
-<contactref element="R15" pad="1"/>
 <contactref element="U1" pad="30"/>
-<wire x1="20.25" y1="22.7" x2="-43.85" y2="-89" width="0" layer="19" extent="1-1"/>
+<contactref element="R23" pad="1"/>
+<contactref element="Q1" pad="1"/>
+<wire x1="-47.85" y1="-92" x2="-51.95" y2="-93" width="0" layer="19" extent="1-1"/>
+<wire x1="20.25" y1="22.7" x2="-47.85" y2="-92" width="0" layer="19" extent="1-1"/>
 </signal>
 <signal name="N$32">
-<contactref element="JP8" pad="1"/>
-<contactref element="Q5" pad="3"/>
-<wire x1="-35" y1="-68" x2="-47" y2="-86.9" width="0" layer="19" extent="1-1"/>
+<contactref element="D3" pad="2"/>
+<contactref element="Q1" pad="3"/>
+<wire x1="-51" y1="-90.9" x2="-53.85" y2="-91" width="0" layer="19" extent="1-1"/>
 </signal>
 <signal name="N$29">
-<contactref element="Q5" pad="1"/>
-<contactref element="R15" pad="2"/>
-<contactref element="R23" pad="1"/>
-<wire x1="-47.95" y1="-89.1" x2="-47.85" y2="-92" width="0" layer="19" extent="1-1"/>
-<wire x1="-42.15" y1="-89" x2="-47.95" y2="-89.1" width="0" layer="19" extent="1-1"/>
+<contactref element="D3" pad="1"/>
+<contactref element="JP3" pad="1"/>
+<wire x1="-56.15" y1="-91" x2="-55" y2="-97" width="0" layer="19" extent="1-1"/>
+</signal>
+<signal name="VDD">
+<contactref element="JP3" pad="3"/>
+</signal>
+<signal name="SD_CS">
+<contactref element="SD1" pad="2"/>
+<contactref element="U1" pad="58"/>
+<wire x1="23.75" y1="11.3" x2="-64.85" y2="-79.5" width="0" layer="19" extent="1-1"/>
+</signal>
+<signal name="SD_MOSI">
+<contactref element="SD1" pad="3"/>
+<contactref element="U1" pad="57"/>
+<wire x1="23.25" y1="11.3" x2="-65.95" y2="-79.5" width="0" layer="19" extent="1-1"/>
+</signal>
+<signal name="SD_CLK">
+<contactref element="SD1" pad="5"/>
+<contactref element="U1" pad="55"/>
+<wire x1="22.25" y1="11.3" x2="-68.15" y2="-79.5" width="0" layer="19" extent="1-1"/>
+</signal>
+<signal name="SD_MISO">
+<contactref element="SD1" pad="7"/>
+<contactref element="U1" pad="56"/>
+<wire x1="22.75" y1="11.3" x2="-70.35" y2="-79.5" width="0" layer="19" extent="1-1"/>
 </signal>
 </signals>

Commit message: update pcb
Parts:
- removed JP5: M02PTH, SparkFun-Connectors:1X02
- removed R9: 20K, SparkFun-Resistors:1206
- removed U$1: SPI_FLASH-X25XXSMD, SparkFun-DigitalIC:SO08
- added R15: 20K, SparkFun-Passives:0603-RES
- added TP1, TP2: TEST-POINT3X5, SparkFun-Passives:PAD.03X.05
- added U2: SPI_FLASH-X25XXSMD, SparkFun-DigitalIC:SO08
- F1: value (none) -> 5V 500mA
- IC5: value (none) -> XC6206
- JP3: value (none) -> LCD_SOCKET
- JP6: value (none) -> USART1
- JP7: value (none) -> SWD
- R1, R2: device SparkFun-Resistors:1206 -> SparkFun-Passives:0603-RES
- S4: value (none) -> POWER
- moved JP3 168.4 mm to (35.5, 45.0), turned to 180 degrees
- moved D3 158.7 mm to (31.5, 42.0)
- moved R23 154.7 mm to (34.5, 39.5), turned to 270 degrees
- moved Q1 152.0 mm to (26.0, 39.0)
- moved R22 137.3 mm to (33.5, 36.0)
- moved C22 131.1 mm to (26.0, 36.0)
- moved R21 130.4 mm to (30.0, 36.0)
- moved SD1 129.1 mm to (22.5, 0.00), flipped to the bottom
- moved R18 126.6 mm to (20.0, 40.0), turned to 270 degrees
- moved R16 118.1 mm to (2.50, 26.0), turned to 90 degrees
- moved C20 86.8 mm to (18.0, 32.0), flipped to the bottom
- moved C19 82.6 mm to (16.5, 36.5), turned to 90 degrees
- moved R13 81.5 mm to (18.0, 29.0), flipped to the bottom
- moved C6 75.2 mm to (15.0, 40.0)
- moved JP2 74.6 mm to (8.00, 46.0)
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Connections:
- removed net IR_EMITTER: IC1.1
- removed net VDD: JP3.3
- net 3.3V: now also JP3.3, TP1.P$1, U2.8; no longer JP5.1, U$1.8
- net AUDIO_ENABLE: now also U1.37
- net FLASH_CLK: now also U2.6; no longer U$1.6
- net FLASH_CS: now also U2.1; no longer U$1.1
- net FLASH_MISO: now also U2.2; no longer U$1.2
- net FLASH_MOSI: now also U2.5; no longer U$1.5
- net GND: now also U2.4; no longer U$1.4
- net IR_EMMITER: now also IC1.1
- net N$14: now also U1.26
- net N$18: now also R15.2; no longer R2.1
- net N$19: now also R2.1; no longer R9.1
- net N$2: now also TP2.P$1; no longer JP5.2
- net N$21: now also R15.1; no longer R9.2
- net N$26: now also U2.3, U2.7; no longer U$1.3, U$1.7
Routing:
- net GND: track 406.5 -> 26.9 mm, vias 67 -> 0
- net 3.3V: track 85.2 -> 5.04 mm, vias 6 -> 0
- net BTN_RELOAD: track 53.8 -> 0.00 mm, vias 2 -> 0
- net BTN_FIRE: track 37.2 -> 0.00 mm
- net 5V: track 152.3 -> 117.3 mm, vias 4 -> 3
- net V_BATT: track 0.00 -> 22.3 mm
- net N$2: track 20.0 -> 0.00 mm, vias 1 -> 0
- net N$8: track 15.8 -> 0.00 mm
- net IR_EMITTER: track 10.3 -> 0.00 mm, vias 1 -> 0
- net SWDIO: track 9.34 -> 0.00 mm, vias 2 -> 0
- net SWDCLK: track 8.60 -> 0.00 mm
- net N$4: track 8.47 -> 0.00 mm, vias 1 -> 0
- net N$3: track 8.47 -> 0.00 mm, vias 1 -> 0
- net N$40: track 7.89 -> 0.00 mm
- net N$44: track 7.17 -> 0.00 mm
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Other:
- board size 72 x 45 mm -> 72 x 50 mm
